Commit message: Add cube detection and overlay nodes
- Implemented the cube detection node in `cube_detector_node.cpp`, which initializes and spins the cube detector.
- Removed the old cube detection node implementation.
- Created a new detection overlay node in `detection_overlay_node.cpp`, responsible for overlaying detection results on images.
- Added the main functionality for the detection overlay in `detection_overlay.cpp`, including image subscription, detection handling, and image publishing with overlays.

File: software/ros_ws/src/perseus_description/urdf/perseus.urdf.xacro (robot description, xacro)
@@ -49,4 +49,16 @@
     <xacro:property name="livox_radius" value="0.04"/>
     <xacro:property name="livox_length" value="0.04"/>
+    <!-- Sensor Mount Properties -->
+    <xacro:property name="sensor_mount_mass" value="0.3"/>
+    <xacro:property name="sensor_mount_length" value="0.08"/>
+    <xacro:property name="sensor_mount_width" value="0.15"/>
+    <xacro:property name="sensor_mount_height" value="0.06"/>
+    <!-- chassis origin is the centre of its front face at the bottom, so x near 0 is the
+         front and z above chassis_height clears the deck -->
+    <xacro:property name="sensor_mount_x_offset" value="0.0"/>
+    <xacro:property name="sensor_mount_y_offset" value="0.0"/>
+    <xacro:property name="sensor_mount_z_offset" value="${chassis_height + 0.05}"/>
+    <!-- nose-down tilt of the Livox: positive pitch swings its +x axis towards -z -->
+    <xacro:property name="livox_pitch" value="${pi/4}"/>
     <!-- ADD COMPONENTS -->
     <xacro:include filename="$(find perseus_description)/urdf/inertia_macros.xacro"/>
@@ -57,4 +69,5 @@
     <xacro:include filename="$(find perseus_description)/urdf/rocker.urdf.xacro"/>
     <xacro:include filename="$(find perseus_description)/urdf/sensors.urdf.xacro"/>
+    <xacro:include filename="$(find perseus_description)/urdf/sensor_mount.urdf.xacro"/>
     <xacro:include filename="$(find perseus_description)/urdf/camera_d455_gazebo.xacro"/>
     <xacro:include filename="$(find realsense2_description)/urdf/_d455.urdf.xacro"/>
@@ -80,9 +93,6 @@
       <child link="${prefix}flange_bearing"/>
     </joint>
-    <joint name="${prefix}laser_joint" type="fixed">
-      <parent link="${prefix}chassis"/>
-      <child link="${prefix}livox_frame"/>
-      <origin xyz="-0.173 0.047 -0.04375" rpy="0 ${pi} ${pi/2}"/>
-    </joint>
+    <!-- Livox and RealSense both hang off the mast: see sensor_mount.urdf.xacro -->
+    <xacro:sensor_mount prefix="${prefix}"/>
     <joint name="${prefix}laser_2d_joint" type="fixed">
       <parent link="${prefix}chassis"/>
@@ -90,8 +100,4 @@
       <origin xyz="-0.15 0 0.25" rpy="0 0 0"/>
     </joint>
-    <xacro:sensor_d455 parent="${prefix}chassis" name="camera" use_nominal_extrinsics="true">
-      <origin xyz="0.055 0.0 0.184" rpy="0 0 0"/>
-    </xacro:sensor_d455>
-    <xacro:camera_d455_gazebo name="camera"/>
   </xacro:macro>
 </robot>
