Commit message: Implement new feature for user authentication and improve error handling

File: software/ros_ws/src/perseus_description/urdf/sensor_mount.urdf.xacro (robot description, xacro)
@@ -17,4 +17,10 @@
         <xacro:box_inertia m="${sensor_mount_mass}" x="${sensor_mount_length}" y="${sensor_mount_width}" z="${sensor_mount_height}"/>
       </inertial>
+      <visual>
+        <origin xyz="0.0 0.0 0.0" rpy="0.0 0.0 ${pi/2}"/>
+        <geometry>
+          <mesh scale="1.0 1.0 1.0" filename="file://$(find perseus_description)/meshes/sensor_mount.dae"/>
+        </geometry>
+      </visual>
     </link>
     <joint name="${prefix}sensor_mount_joint" type="fixed">

File: software/ros_ws/src/perseus_description/urdf/sensors.urdf.xacro (robot description, xacro)
@@ -13,5 +13,4 @@
             <mesh scale="1.0 1.0  1.0" filename="file://$(find perseus_description)/meshes/mid-360.dae"/>
         </geometry>
-        <material name="black"/>
     </visual>
     <collision>

Commit message: Fix sensor_mount visual origin offset for improved alignment:

File: software/ros_ws/src/perseus_description/urdf/sensor_mount.urdf.xacro (robot description, xacro)
@@ -18,5 +18,5 @@
       </inertial>
       <visual>
-        <origin xyz="0.0 0.0 0.0" rpy="0.0 0.0 ${pi/2}"/>
+        <origin xyz="0.0 0.0 ${-0.04}" rpy="0.0 0.0 ${pi/2}"/>
         <geometry>
           <mesh scale="1.0 1.0 1.0" filename="file://$(find perseus_description)/meshes/sensor_mount.dae"/>

Commit message: Adjust sensor_mount visual origin offsets for improved alignment

File: software/ros_ws/src/perseus_description/urdf/sensor_mount.urdf.xacro (robot description, xacro)
@@ -18,5 +18,5 @@
       </inertial>
       <visual>
-        <origin xyz="0.0 0.0 ${-0.04}" rpy="0.0 0.0 ${pi/2}"/>
+        <origin xyz="${-0.023} ${0.01} ${-0.035}" rpy="0.0 0.0 ${pi/2}"/>
         <geometry>
           <mesh scale="1.0 1.0 1.0" filename="file://$(find perseus_description)/meshes/sensor_mount.dae"/>
@@ -42,5 +42,5 @@
     <!-- RealSense D455, on the front face of the mast, looking straight ahead -->
     <xacro:sensor_d455 parent="${prefix}sensor_mount" name="camera" use_nominal_extrinsics="true">
-      <origin xyz="0.0 0.0 0.0" rpy="0.0 0.0 0.0"/>
+      <origin xyz="0.035 0.0 0.006" rpy="0.0 0.0 0.0"/>
     </xacro:sensor_d455>
     <xacro:camera_d455_gazebo name="camera"/>

Commit message: Adjust sensor_mount visual origin offsets for improved alignment

File: software/ros_ws/src/perseus_description/urdf/sensor_mount.urdf.xacro (robot description, xacro)
@@ -18,5 +18,5 @@
       </inertial>
       <visual>
-        <origin xyz="${-0.023} ${0.01} ${-0.035}" rpy="0.0 0.0 ${pi/2}"/>
+        <origin xyz="${-0.023} ${0.005} ${-0.035}" rpy="0.0 0.0 ${pi/2}"/>
         <geometry>
           <mesh scale="1.0 1.0 1.0" filename="file://$(find perseus_description)/meshes/sensor_mount.dae"/>
@@ -38,5 +38,5 @@
       <parent link="${prefix}sensor_mount"/>
       <child link="${prefix}livox_frame"/>
-      <origin xyz="0.0 0.0 0.1" rpy="0.0 ${livox_pitch} 0.0"/>
+      <origin xyz="0.04 0.0 0.13" rpy="0.0 ${livox_pitch} 0.0"/>
     </joint>
     <!-- RealSense D455, on the front face of the mast, looking straight ahead -->
