File: hardware/enc-encoder/RS485.kicad_sch (KiCad schematic)
At the start: 5 parts, among them U4 SP3485CN

Commit message: Feat: Updated sheet names and titles
Other:
- title: (none) -> RS485 Slave
Changed lines of the file:
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@@
 	(generator_version "10.0")
 	(paper "A4")
+	(title_block
+		(title "RS485 Slave")
+		(date "2026-08-15")
+		(rev "V1R1")
+	)
 	(text "0.25 W"
 		(exclude_from_sim no)
