File: hardware/enc-encoder/enc-encoder.kicad_sch (KiCad schematic)
At the start: 43 parts, among them J1 OQ0232510000G, J2 OQ0232510000G, J3 USB_C_Receptacle, J4 SM03B-SRSS-TB, J5 OQ0232510000G, J6 OQ0232510000G, SW1 219-4LPSTR, U3 AS5600

Commit message: Feat: Finished Encoder PCB Routing
Finished PCB routing for the EnC magnetic encoder. Some minor improvements and fabrication markings still needed
Parts:
- 3V1, GND1, VBUS1, VCC1: footprint TestPoint:TestPoint_Pad_D2.0mm -> TestPoint:TestPoint_Pad_D1.0mm
Connections:
- net +3.3V: now also R8.2; no longer SW1.8, U3.8 (DIR)
- net GND: now also SW1.1; no longer R8.1
- new net HALL_DIR: R8.1, SW1.8, U3.8 (DIR)
Other:
- moved on the sheet: R8
Changed lines of the file:
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@@
 	(wire
 		(pts
-			(xy 99.06 175.26) (xy 100.33 175.26)
+			(xy 99.06 175.26) (xy 107.95 175.26)
 		)
 		(stroke
@@
 	(symbol
 		(lib_id "Device:R")
-		(at 104.14 175.26 90)
+		(at 123.19 167.64 180)
 		(unit 1)
 		(body_style 1)
@@
 		(dnp no)
 		(property "Reference" "R8"
-			(at 103.124 172.212 90)
+			(at 120.142 168.656 90)
 			(show_name no)
 			(do_not_autoplace no)
@@
 		)
 		(property "Value" "10k"
-			(at 107.442 172.212 90)
+			(at 120.142 164.338 90)
 			(show_name no)
 			(do_not_autoplace no)
@@
 		)
 		(property "Footprint" "Resistor_SMD:R_0603_1608Metric_Pad0.98x0.95mm_HandSolder"
-			(at 104.14 177.038 90)
+			(at 124.968 167.64 90)
 			(hide yes)
 			(show_name no)
@@
 		)
 		(property "Datasheet" "https://yageogroup.com/content/datasheet/asset/file/PYU-RC_GROUP_51_ROHS_L"
-			(at 104.14 175.26 0)
+			(at 123.19 167.64 0)
 			(hide yes)
 			(show_name no)
@@
 		)
 		(property "Description" "Resistor"
-			(at 104.14 175.26 0)
+			(at 123.19 167.64 0)
 			(hide yes)
 			(show_name no)
@@
 		)
 		(property "Supplier" "DigiKey"
-			(at 104.14 175.26 0)
+			(at 123.19 167.64 0)
 			(hide yes)
 			(show_name no)
@@
 		)
 		(property "Supplier Link" "https://www.digikey.com.au/en/products/detail/yageo/RC0603FR-0710KL/726880"
-			(at 104.14 175.26 0)
+			(at 123.19 167.64 0)
 			(hide yes)
 			(show_name no)
@@
 		)
 		(property "Supplier Part No" "311-10.0KHRCT-ND"
-			(at 104.14 175.26 0)
+			(at 123.19 167.64 0)
 			(hide yes)
 			(show_name no)
@@
 		)
 		(property "KLC_S4.2_DVDD" ""
-			(at 104.14 175.26 0)
+			(at 123.19 167.64 0)
 			(hide yes)
 			(show_name no)
@@
 		)
 		(property "KLC_S4.2_VREG_LX" ""
-			(at 104.14 175.26 0)
+			(at 123.19 167.64 0)
 			(hide yes)
 			(show_name no)
@@
 		)
 		(property "KLC_S3.3" ""
-			(at 104.14 175.26 0)
+			(at 123.19 167.64 0)
 			(hide yes)
 			(show_name no)
@@
 		)
 		(property "KLC_S4.1" ""
-			(at 104.14 175.26 0)
+			(at 123.19 167.64 0)
 			(hide yes)
 			(show_name no)
@@
 	)
 	(symbol
+		(lib_id "power:+3.3V")
+		(at 123.19 163.83 0)
+		(unit 1)
+		(body_style 1)
+		(exclude_from_sim no)
+		(in_bom yes)
+		(on_board yes)
+		(in_pos_files yes)
+		(dnp no)
+		(fields_autoplaced yes)
+		(property "Reference" "#PWR08"
+			(at 123.19 167.64 0)
+			(hide yes)
+			(show_name no)
+			(do_not_autoplace no)
+			(effects
+				(font
+					(size 1.27 1.27)
+				)
+			)
+		)
+		(property "Value" "+3.3V"
+			(at 123.19 158.75 0)
+			(show_name no)
+			(do_not_autoplace no)
+			(effects
+				(font
+					(size 1.27 1.27)
+				)
+			)
+		)
+		(property "Footprint" ""
+			(at 123.19 163.83 0)
+			(hide yes)
+			(show_name no)
+			(do_not_autoplace no)
+			(effects
+				(font
+					(size 1.27 1.27)
+				)
+			)
+		)
+		(property "Datasheet" ""
+			(at 123.19 163.83 0)
+			(hide yes)
+			(show_name no)
+			(do_not_autoplace no)
+			(effects
+				(font
+					(size 1.27 1.27)
+				)
+			)
+		)
+		(property "Description" "Power symbol creates a global label with name \"+3.3V\""
+			(at 123.19 163.83 0)
+			(hide yes)
+			(show_name no)
+			(do_not_autoplace no)
+			(effects
+				(font
+					(size 1.27 1.27)
+				)
+			)
+		)
+		(pin "1"
+		)
+		(instances
+			(project "enc-encoder"
+				(path "/830e855f-c01b-4865-ac3f-fca5cbe32ffd"
+					(reference "#PWR08")
+					(unit 1)
+				)
+			)
+		)
+	)
+	(symbol
 		(lib_id "Connector_Generic:Conn_01x02")
 		(at 41.91 40.64 0)
@@
 			)
 		)
-		(property "Footprint" "TestPoint:TestPoint_Pad_D2.0mm"
+		(property "Footprint" "TestPoint:TestPoint_Pad_D1.0mm"
 			(at 259.08 154.94 0)
 			(hide yes)
@@
 			)
 		)
-		(property "Footprint" "TestPoint:TestPoint_Pad_D2.0mm"
+		(property "Footprint" "TestPoint:TestPoint_Pad_D1.0mm"
 			(at 180.34 134.62 0)
 			(hide yes)
@@
 			)
 		)
-		(property "Footprint" "TestPoint:TestPoint_Pad_D2.0mm"
+		(property "Footprint" "TestPoint:TestPoint_Pad_D1.0mm"
 			(at 248.92 167.64 0)
 			(hide yes)
@@
 	)
 	(symbol
-		(lib_id "power:+3.3V")
-		(at 123.19 171.45 0)
-		(unit 1)
-		(body_style 1)
-		(exclude_from_sim no)
-		(in_bom yes)
-		(on_board yes)
-		(in_pos_files yes)
-		(dnp no)
-		(property "Reference" "#PWR08"
-			(at 123.19 175.26 0)
-			(hide yes)
-			(show_name no)
-			(do_not_autoplace no)
-			(effects
-				(font
-					(size 1.27 1.27)
-				)
-			)
-		)
-		(property "Value" "+3.3V"
-			(at 123.19 167.64 0)
-			(show_name no)
-			(do_not_autoplace no)
-			(effects
-				(font
-					(size 1.27 1.27)
-				)
-			)
-		)
-		(property "Footprint" ""
-			(at 123.19 171.45 0)
-			(hide yes)
-			(show_name no)
-			(do_not_autoplace no)
-			(effects
-				(font
-					(size 1.27 1.27)
-				)
-			)
-		)
-		(property "Datasheet" ""
-			(at 123.19 171.45 0)
-			(hide yes)
-			(show_name no)
-			(do_not_autoplace no)
-			(effects
-				(font
-					(size 1.27 1.27)
-				)
-			)
-		)
-		(property "Description" "Power symbol creates a global label with name \"+3.3V\""
-			(at 123.19 171.45 0)
-			(hide yes)
-			(show_name no)
-			(do_not_autoplace no)
-			(effects
-				(font
-					(size 1.27 1.27)
-				)
-			)
-		)
-		(pin "1"
-		)
-		(instances
-			(project "enc-encoder"
-				(path "/830e855f-c01b-4865-ac3f-fca5cbe32ffd"
-					(reference "#PWR08")
-					(unit 1)
-				)
-			)
-		)
-	)
-	(symbol
 		(lib_id "power:GND")
 		(at 219.71 152.4 0)
@@
 			)
 		)
-		(property "Footprint" "TestPoint:TestPoint_Pad_D2.0mm"
+		(property "Footprint" "TestPoint:TestPoint_Pad_D1.0mm"
 			(at 222.25 22.86 0)
 			(hide yes)

Commit message: Feat: Fixed USB High-speed trace matching
Fixed USB trace length matching for high-speed data communications.
Connections:
- net RP_HSTX_D0-: now reaches J3.A10 (RX2-)
- net RP_HSTX_D0+: now reaches J3.A11 (RX2+)
- net RP_HSTX_D2+: now reaches J3.A2 (TX1+)
- net RP_HSTX_D2-: now reaches J3.A3 (TX1-)
- net RP_HSTX_CK+: now reaches J3.B10 (RX1-)
- net RP_HSTX_CK-: now reaches J3.B11 (RX1+)
- net RP_HSTX_D1+: now reaches J3.B2 (TX2+)
- net RP_HSTX_D1-: now reaches J3.B3 (TX2-)
- no-connect marks 11 -> 3
Other:
- sheet rp2350 ports: added RP_HSTX_CK+, RP_HSTX_CK-, RP_HSTX_D0+, RP_HSTX_D0-, RP_HSTX_D1+, RP_HSTX_D1-, RP_HSTX_D2+, RP_HSTX_D2-; removed none
- moved on the sheet: D1

Commit message: Feat: Added Silkscreen Indicators
Parts:
- renumbered 3V1 to 3V3
Changed lines of the file:
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@@
 		(in_pos_files yes)
 		(dnp no)
-		(property "Reference" "3V1"
+		(property "Reference" "3V3"
 			(at 252.222 150.622 0)
 			(show_name no)
@@
 			(project "enc-encoder"
 				(path "/830e855f-c01b-4865-ac3f-fca5cbe32ffd"
-					(reference "3V1")
+					(reference "3V3")
 					(unit 1)
 				)
