File: hardware/enc-encoder/RS485_slave.kicad_sch (KiCad schematic)
At the start: 5 parts, among them U4 SP3485CN

Commit message: added fiducials for PNP and silkscreen
Other:
- title: RS485 Slave -> Magnetic Angle Sensor
Changed lines of the file:
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@@
 	(paper "A4")
 	(title_block
-		(title "RS485 Slave")
-		(date "2026-08-15")
+		(title "Magnetic Angle Sensor")
+		(date "2026-08-25")
 		(rev "V1R1")
 	)
