File: hardware/dc-motor-driver/RS485.kicad_sch (KiCad schematic)
At the start: 7 parts, among them J10 ECH350R-04P, U7 SP3485CN

Commit message: Feat: Finished PCB for review
Fixed RS485 connectors, finished traces and PCB layout. Ready for review before manufacturing
Parts:
- removed J10: ECH350R-04P, ConnectorsOther:TerminalBlock_Dinkle_ECH350R-04_P3.50mm, symbol Connector_Generic:Conn_01x04
- added J10, J11: OQ0232510000G, ConnectorsOther:AnyTek_OQ_3.81mm_90_2P_TriangleKeyLock, symbol Connector_Generic:Conn_01x02
Connections:
- net +3V3: now also J10.1 (Pin_1)
- net GND: now also J10.2 (Pin_2)
- net A: no longer names the net of D1.2 (A2), R16.2, R17.1, U7.6 (A)
- net A: now also J11.1 (Pin_1)
- net B: no longer names the net of D1.1 (A1), R17.2, R18.1, U7.7 (B)
- net B: now also J11.2 (Pin_2)

Commit message: Fix: PCB, schematic errors
Added M8 footprint and wiring. Fixed silkscreen issues and RS485 power out (now 24V)
Connections:
- net +3V3: no longer J10.1 (Pin_1)
- new net VCC: J10.1 (Pin_1)
Changed lines of the file:
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@@
+	)
+	(symbol
+		(lib_id "power:VCC")
+		(at 162.56 74.93 0)
+		(unit 1)
+		(body_style 1)
+		(exclude_from_sim no)
+		(in_bom yes)
+		(on_board yes)
+		(in_pos_files yes)
+		(dnp no)
+		(property "Reference" "#PWR068"
+			(at 162.56 78.74 0)
+			(hide yes)
+			(show_name no)
+			(do_not_autoplace no)
+			(effects
+				(font
+					(size 1.27 1.27)
+				)
+			)
+		)
+		(property "Value" "VCC"
+			(at 162.56 71.12 0)
+			(show_name no)
+			(do_not_autoplace no)
+			(effects
+				(font
+					(size 1.27 1.27)
+				)
+			)
+		)
+		(property "Footprint" ""
+			(at 162.56 74.93 0)
+			(hide yes)
+			(show_name no)
+			(do_not_autoplace no)
+			(effects
+				(font
+					(size 1.27 1.27)
+				)
+			)
+		)
+		(property "Datasheet" ""
+			(at 162.56 74.93 0)
+			(hide yes)
+			(show_name no)
+			(do_not_autoplace no)
+			(effects
+				(font
+					(size 1.27 1.27)
+				)
+			)
+		)
+		(property "Description" "Power symbol creates a global label with name \"VCC\""
+			(at 162.56 74.93 0)
+			(hide yes)
+			(show_name no)
+			(do_not_autoplace no)
+			(effects
+				(font
+					(size 1.27 1.27)
+				)
+			)
+		)
+		(pin "1"
+		)
+		(instances
+			(project "dc-motor-driver"
+				(path "/fc286157-4263-4a46-ad05-98b3354aa28a/248c9f41-6be5-4998-8da0-57ff13dead05"
+					(reference "#PWR068")
+					(unit 1)
+				)
+				(path "/fc286157-4263-4a46-ad05-98b3354aa28a/61fde4a3-9ead-4a32-9461-24e8bd358e08"
+					(reference "#PWR075")
+					(unit 1)
+				)
+			)
+		)
 	)
 	(symbol
@@
 					(unit 1)
 				)
-			)
-		)
-	)
-	(symbol
-		(lib_id "power:+3V3")
-		(at 162.56 74.93 0)
-		(unit 1)
-		(body_style 1)
-		(exclude_from_sim no)
-		(in_bom yes)
-		(on_board yes)
-		(in_pos_files yes)
-		(dnp no)
-		(property "Reference" "#PWR068"
-			(at 162.56 78.74 0)
-			(hide yes)
-			(show_name no)
-			(do_not_autoplace no)
-			(effects
-				(font
-					(size 1.27 1.27)
-				)
-			)
-		)
-		(property "Value" "+3V3"
-			(at 162.56 71.12 0)
-			(show_name no)
-			(do_not_autoplace no)
-			(effects
-				(font
-					(size 1.27 1.27)
-				)
-			)
-		)
-		(property "Footprint" ""
-			(at 162.56 74.93 0)
-			(hide yes)
-			(show_name no)
-			(do_not_autoplace no)
-			(effects
-				(font
-					(size 1.27 1.27)
-				)
-			)
-		)
-		(property "Datasheet" ""
-			(at 162.56 74.93 0)
-			(hide yes)
-			(show_name no)
-			(do_not_autoplace no)
-			(effects
-				(font
-					(size 1.27 1.27)
-				)
-			)
-		)
-		(property "Description" "Power symbol creates a global label with name \"+3V3\""
-			(at 162.56 74.93 0)
-			(hide yes)
-			(show_name no)
-			(do_not_autoplace no)
-			(effects
-				(font
-					(size 1.27 1.27)
-				)
-			)
-		)
-		(pin "1"
-		)
-		(instances
-			(project "RS485"
-				(path "/2d7ae3dd-bfc0-4939-b7a9-b7e986e3c078"
-					(reference "#PWR068")
-					(unit 1)
-				)
-			)
-			(project "dc-motor-driver"
-				(path "/fc286157-4263-4a46-ad05-98b3354aa28a/248c9f41-6be5-4998-8da0-57ff13dead05"
-					(reference "#PWR068")
-					(unit 1)
-				)
-				(path "/fc286157-4263-4a46-ad05-98b3354aa28a/61fde4a3-9ead-4a32-9461-24e8bd358e08"
-					(reference "#PWR075")
-					(unit 1)
-				)

Commit message: Feat: Fixed sheet names and BOM
Fixed missing values from BOM. Added correct title and revision to sheet details
Parts:
- J11: Supplier (none) -> DigiKey; Supplier Link (none) -> https://www.digikey.com/en/products/detail/amphenol-anytek/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; Supplier Part No (none) -> 609-3819-ND
Other:
- title: (none) -> RS485 Master
Changed lines of the file:
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@@
 	(generator_version "10.0")
 	(paper "A4")
+	(title_block
+		(title "RS485 Master")
+		(date "2026-08-15")
+		(rev "V1R1")
+	)
 	(text "0.25 W"
 		(exclude_from_sim no)
@@
 			(at 170.18 81.28 0)
 			(hide yes)
+			(show_name no)
+			(do_not_autoplace no)
+			(effects
+				(font
+					(size 1.27 1.27)
+				)
+			)
+		)
+		(property "Supplier" "DigiKey"
+			(at 170.18 81.28 0)
+			(hide yes)
+			(show_name no)
+			(do_not_autoplace no)
+			(effects
+				(font
+					(size 1.27 1.27)
+				)
+			)
+		)
+		(property "Supplier Link" "https://www.digikey.com/en/products/detail/amphenol-anytek/OQ0232510000G/2261255"
+			(at 170.18 81.28 0)
+			(hide yes)
+			(show_name no)
+			(do_not_autoplace no)
+			(effects
+				(font
+					(size 1.27 1.27)
+				)
+			)
+		)
+		(property "Supplier Part No" "609-3819-ND"
+			(at 170.18 81.28 0)
+			(hide yes)
