File: hardware/dc-motor-driver/motor-driver.kicad_sch (KiCad schematic)
At the start: 9 parts, among them J4 MOT, U1 DRV8874PWPR

Commit message: fixed footprint library and changed connectors
Parts:
- removed J4: MOT, TerminalBlock_4Ucon:TerminalBlock_4Ucon_1x02_P3.50mm_Horizontal, symbol Connector:Screw_Terminal_01x02
- added J15: OQ0232510000G, ConnectorsOther:AnyTek_OQ_3.81mm_90_2P_TriangleKeyLock, symbol Connector_Generic:Conn_01x02
Connections:
- net at U1.10 (OUT2): now also J15.1 (Pin_1)
- net at U1.8 (OUT1): now also J15.2 (Pin_2)
Changed lines of the file:
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@@
+	(wire
+		(pts
+			(xy 119.38 25.4) (xy 123.19 25.4)
+		)
+		(stroke
+			(width 0)
+			(type default)
+		)
+	)
 	(wire
 		(pts
@@
 	(wire
 		(pts
-			(xy 121.92 25.4) (xy 119.38 25.4)
+			(xy 73.66 59.69) (xy 73.66 50.8)
 		)
 		(stroke
@@
 	(wire
 		(pts
-			(xy 73.66 59.69) (xy 73.66 50.8)
+			(xy 119.38 27.94) (xy 123.19 27.94)
 		)
 		(stroke
@@
 		(pts
 			(xy 82.55 40.64) (xy 83.82 40.64)
-		)
-		(stroke
-			(width 0)
-			(type default)
-		)
-	)
-	(wire
-		(pts
-			(xy 121.92 27.94) (xy 119.38 27.94)
 		)
 		(stroke
@@
 	)
 	(symbol
+		(lib_id "Connector_Generic:Conn_01x02")
+		(at 128.27 27.94 0)
+		(mirror x)
+		(unit 1)
+		(body_style 1)
+		(exclude_from_sim no)
+		(in_bom yes)
+		(on_board yes)
+		(in_pos_files yes)
+		(dnp no)
+		(property "Reference" "J15"
+			(at 130.81 27.9401 0)
+			(show_name no)
+			(do_not_autoplace no)
+			(effects
+				(font
+					(size 1.27 1.27)
+				)
+				(justify left)
+			)
+		)
+		(property "Value" "OQ0232510000G"
+			(at 130.81 25.4001 0)
+			(show_name no)
+			(do_not_autoplace no)
+			(effects
+				(font
+					(size 1.27 1.27)
+				)
+				(justify left)
+			)
+		)
+		(property "Footprint" "ConnectorsOther:AnyTek_OQ_3.81mm_90_2P_TriangleKeyLock"
+			(at 128.27 27.94 0)
+			(hide yes)
+			(show_name no)
+			(do_not_autoplace no)
+			(effects
+				(font
+					(size 1.27 1.27)
+				)
+			)
+		)
+		(property "Datasheet" "http://www.anytek.com.tw/UserUpFiles/20181018/_S_eBwgMo_mC.pdf"
+			(at 128.27 27.94 0)
+			(hide yes)
+			(show_name no)
+			(do_not_autoplace no)
+			(effects
+				(font
+					(size 1.27 1.27)
+				)
+			)
+		)
+		(property "Description" "Generic connector, single row, 01x02, script generated (kicad-library-utils/schlib/autogen/connector/)"
+			(at 128.27 27.94 0)
+			(hide yes)
+			(show_name no)
+			(do_not_autoplace no)
+			(effects
+				(font
+					(size 1.27 1.27)
+				)
+			)
+		)
+		(property "Supplier" "DigiKey"
+			(at 128.27 27.94 0)
+			(hide yes)
+			(show_name no)
+			(do_not_autoplace no)
+			(effects
+				(font
+					(size 1.27 1.27)
+				)
+			)
+		)
+		(property "Supplier Part No" "609-3819-ND"
+			(at 128.27 27.94 0)
+			(hide yes)
+			(show_name no)
+			(do_not_autoplace no)
+			(effects
+				(font
+					(size 1.27 1.27)
+				)
+			)
+		)
+		(property "Supplier Link" "https://www.digikey.com/en/products/detail/amphenol-anytek/OQ0232510000G/2261255"
+			(at 128.27 27.94 0)
+			(hide yes)
+			(show_name no)
+			(do_not_autoplace no)
+			(effects
+				(font
+					(size 1.27 1.27)
+				)
+			)
+		)
+		(pin "1"
+		)
+		(pin "2"
+		)
+		(instances
+			(project "dc-motor-driver"
+				(path "/fc286157-4263-4a46-ad05-98b3354aa28a/40f5114d-d621-443c-9e87-66cb3392bce6"
+					(reference "J18")
+					(unit 1)
+				)
+				(path "/fc286157-4263-4a46-ad05-98b3354aa28a/47ca5528-118a-41e5-93e9-251f6cf35694"
+					(reference "J19")
+					(unit 1)
+				)
+				(path "/fc286157-4263-4a46-ad05-98b3354aa28a/7de317d4-3d1e-4d6a-9df4-d39eb3e35b32"
+					(reference "J15")
+					(unit 1)
+				)
+				(path "/fc286157-4263-4a46-ad05-98b3354aa28a/92e3a97b-4604-4305-8719-7a31c2be7d8e"
+					(reference "J16")
+					(unit 1)
+				)
+				(path "/fc286157-4263-4a46-ad05-98b3354aa28a/cb7f55f2-47ab-49cc-bc72-89df683d7d50"
+					(reference "J17")
+					(unit 1)
+				)
+				(path "/fc286157-4263-4a46-ad05-98b3354aa28a/d9a6d9bc-65d3-41fc-becf-b57a61750c4d"
+					(reference "J20")
+					(unit 1)
+				)
+			)
+		)
+	)
+	(symbol
 		(lib_id "power:GND")
 		(at 101.6 63.5 0)
@@
 					(unit 1)
 				)
-			)
-		)
-	)
-	(symbol
-		(lib_id "Connector:Screw_Terminal_01x02")
-		(at 127 25.4 0)
-		(unit 1)
-		(body_style 1)
-		(exclude_from_sim no)
-		(in_bom yes)
-		(on_board yes)
-		(in_pos_files yes)
-		(dnp no)
-		(property "Reference" "J4"
-			(at 130.175 25.3999 0)
-			(show_name no)
-			(do_not_autoplace no)
-			(effects
-				(font
-					(size 1.27 1.27)
-				)
-				(justify left)
-			)
-		)
-		(property "Value" "MOT"
-			(at 130.175 27.9399 0)
-			(show_name no)
-			(do_not_autoplace no)
-			(effects
-				(font
-					(size 1.27 1.27)
-				)
-				(justify left)
-			)
-		)
-		(property "Footprint" "TerminalBlock_4Ucon:TerminalBlock_4Ucon_1x02_P3.50mm_Horizontal"
-			(at 127 25.4 0)
-			(hide yes)
-			(show_name no)
-			(do_not_autoplace no)
-			(effects
-				(font
-					(size 1.27 1.27)
-				)
-			)
-		)
-		(property "Datasheet" ""
-			(at 127 25.4 0)
-			(hide yes)
-			(show_name no)
-			(do_not_autoplace no)
-			(effects
-				(font
-					(size 1.27 1.27)
-				)
-			)
-		)
-		(property "Description" "Generic screw terminal, single row, 01x02, script generated (kicad-library-utils/schlib/autogen/connector/)"
-			(at 127 25.4 0)
-			(hide yes)
-			(show_name no)
-			(do_not_autoplace no)
-			(effects
-				(font
-					(size 1.27 1.27)
-				)
-			)
-		)
-		(property "Supplier" ""
-			(at 127 25.4 0)
-			(show_name no)
-			(do_not_autoplace no)
-			(effects
-				(font
-					(size 1.27 1.27)
-				)
-			)
-		)
-		(pin "1"
-		)
-		(pin "2"
-		)
-		(instances
-			(project "dc-motor-driver"
-				(path "/fc286157-4263-4a46-ad05-98b3354aa28a/40f5114d-d621-443c-9e87-66cb3392bce6"
-					(reference "J7")
-					(unit 1)
-				)
-				(path "/fc286157-4263-4a46-ad05-98b3354aa28a/47ca5528-118a-41e5-93e9-251f6cf35694"
-					(reference "J8")
-					(unit 1)
-				)
-				(path "/fc286157-4263-4a46-ad05-98b3354aa28a/7de317d4-3d1e-4d6a-9df4-d39eb3e35b32"
-					(reference "J4")
-					(unit 1)
-				)
-				(path "/fc286157-4263-4a46-ad05-98b3354aa28a/92e3a97b-4604-4305-8719-7a31c2be7d8e"
-					(reference "J5")
-					(unit 1)
-				)
-				(path "/fc286157-4263-4a46-ad05-98b3354aa28a/cb7f55f2-47ab-49cc-bc72-89df683d7d50"
-					(reference "J6")
-					(unit 1)
-				)
-				(path "/fc286157-4263-4a46-ad05-98b3354aa28a/d9a6d9bc-65d3-41fc-becf-b57a61750c4d"
-					(reference "J9")
-					(unit 1)
-				)
