File: hardware/dc-motor-driver/dc-motor-driver.kicad_sch (KiCad schematic)
At the start: 12 parts, among them J1 VIN, J3 DE9

Commit message: Feat: Finished PCB for review
Fixed RS485 connectors, finished traces and PCB layout. Ready for review before manufacturing
Connections:
- net MCU2_DIR: now also PCB1.30 (IO39); no longer PCB1.31 (IO40)
- net ~{SLEEP}: now also PCB1.31 (IO40); no longer PCB1.30 (IO39)
Changed lines of the file:
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@@
 	(wire
 		(pts
-			(xy 142.24 127) (xy 148.59 127)
+			(xy 142.24 124.46) (xy 152.4 124.46)
 		)
 		(stroke
@@
 	(wire
 		(pts
-			(xy 142.24 124.46) (xy 152.4 124.46)
-		)
-		(stroke
-			(width 0)
-			(type default)
-		)
-	)
-	(wire
-		(pts
 			(xy 148.59 33.02) (xy 163.83 33.02)
 		)
@@
 	(wire
 		(pts
+			(xy 142.24 127) (xy 152.4 127)
+		)
+		(stroke
+			(width 0)
+			(type default)
+		)
+	)
+	(wire
+		(pts
 			(xy 142.24 134.62) (xy 152.4 134.62)
 		)
@@
 	)
 	(label "~{SLEEP}"
-		(at 148.59 127 180)
+		(at 152.4 124.46 180)
 		(effects
 			(font
@@
 	)
 	(label "MCU2_DIR"
-		(at 152.4 124.46 180)
-		(effects
-			(font
+		(at 152.4 127 180)
+		(effects
+			(font

Commit message: Fix: PCB, schematic errors
Added M8 footprint and wiring. Fixed silkscreen issues and RS485 power out (now 24V)
Parts:
- removed J1: VIN, TerminalBlock_4Ucon:TerminalBlock_4Ucon_1x02_P3.50mm_Horizontal, symbol Connector:Screw_Terminal_01x02
- removed J2: (no value), Connector_AMASS:AMASS_XT60PW-M_1x02_P7.20mm_Horizontal, symbol Manufacturer_Connectors:XT_Connector
- removed J3: DE9, THT:A-DF_09_A_KG-T2S, symbol Manufacturer_Connectors:A-DF_09_A/KG-T2S
- added J14: 54-00274, ConnectorsOther:Tensility_M8_Socket_4P_Shielded_A, symbol Manufacturer Connectors:54-00274
- added J2: VIN, Connector_AMASS:AMASS_XT60PW-M_1x02_P7.20mm_Horizontal, symbol Manufacturer Connectors:XT_Connector
- added J3: DE9, THT:A-DF_09_A_KG-T2S, symbol Manufacturer Connectors:A-DF_09_A/KG-T2S
Connections:
- net GND: now also J14.S1 (SHIELD), J14.S2 (SHIELD__1), J2.1 (-), J3.0 (PAD)
- net VCC: now also J2.2 (+)
- net CAN+ renamed CAN_H
- net CAN_H: now also J14.2, J3.7, J3.8
- net CAN- renamed CAN_L
- net CAN_L: now also J14.1, J3.1, J3.2
- no-connect marks 14 -> 16

Commit message: added silkscreen
Parts:
- added FID1, FID2, FID3: Fiducial, Fiducial:Fiducial_1.5mm_Mask3mm, symbol Mechanical:Fiducial
Other:
- note added: "Fiducial for PNP"

Commit message: fixed footprint library and changed connectors
Parts:
- J14: now fitted
Changed lines of the file:
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@@
 		(body_style 1)
 		(exclude_from_sim no)
-		(in_bom no)
-		(on_board yes)
-		(in_pos_files yes)
-		(dnp yes)
+		(in_bom yes)
+		(on_board yes)
+		(in_pos_files yes)
+		(dnp no)
 		(fields_autoplaced yes)
 		(property "Reference" "#PWR077"
@@
 		(on_board yes)
 		(in_pos_files yes)
-		(dnp yes)
+		(dnp no)
 		(fields_autoplaced yes)
 		(property "Reference" "J14"

Commit message: manufacture ready
Parts:
- removed J14: 54-00274, ConnectorsOther:Tensility_M8_Socket_4P_Shielded_A, symbol Manufacturer Connectors:54-00274
- added J1: (no value), ConnectorsOther:AnyTek_OQ_3.81mm_90_2P_TriangleKeyLock, symbol ComponentLibrary:anytek_plug_terminal
Connections:
- net CAN_H: now also J1.2
- net CAN_L: now also J1.1
- net GND: now also J1.S1 (SHIELD), J1.S2 (SHIELD__1)
Changed lines of the file:
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@@
+	)
+	(symbol
+		(lib_id "ComponentLibrary:anytek_plug_terminal")
+		(at 58.42 147.32 0)
+		(unit 1)
+		(body_style 1)
+		(exclude_from_sim no)
+		(in_bom yes)
+		(on_board yes)
+		(in_pos_files yes)
+		(dnp no)
+		(fields_autoplaced yes)
+		(property "Reference" "J1"
+			(at 59.055 137.16 0)
+			(show_name no)
+			(do_not_autoplace no)
+			(effects
+				(font
+					(size 1.27 1.27)
+				)
+			)
+		)
+		(property "Value" ""
+			(at 53.34 160.02 0)
+			(hide yes)
+			(show_name no)
+			(do_not_autoplace no)
+			(effects
+				(font
+					(size 1.27 1.27)
+				)
+				(justify left bottom)
+			)
+		)
+		(property "Footprint" "ConnectorsOther:AnyTek_OQ_3.81mm_90_2P_TriangleKeyLock"
+			(at 82.042 160.274 0)
+			(hide yes)
+			(show_name no)
+			(do_not_autoplace no)
+			(effects
+				(font
+					(size 1.27 1.27)
+				)
+				(justify bottom)
+			)
+		)
+		(property "Datasheet" ""
+			(at 58.42 147.32 0)
+			(hide yes)
+			(show_name no)
+			(do_not_autoplace no)
+			(effects
+				(font
+					(size 1.27 1.27)
+				)
+			)
+		)
+		(property "Description" ""
+			(at 58.42 147.32 0)
+			(hide yes)
+			(show_name no)
+			(do_not_autoplace no)
+			(effects
+				(font
+					(size 1.27 1.27)
+				)
+			)
+		)
+		(property "PARTREV" ""
+			(at 54.61 169.672 0)
+			(hide yes)
+			(show_name no)
+			(do_not_autoplace no)
+			(effects
+				(font
+					(size 1.27 1.27)
+				)
+				(justify bottom)
+			)
+		)
+		(property "STANDARD" ""
+			(at 68.834 163.83 0)
+			(hide yes)
+			(show_name no)
+			(do_not_autoplace no)
+			(effects
+				(font
+					(size 1.27 1.27)
+				)
+				(justify bottom)
+			)
+		)
+		(property "MAXIMUM_PACKAGE_HEIGHT" ""
+			(at 58.166 165.608 0)
+			(hide yes)
+			(show_name no)
+			(do_not_autoplace no)
+			(effects
+				(font
+					(size 1.27 1.27)
+				)
+				(justify bottom)
+			)
+		)
+		(property "MANUFACTURER" ""
+			(at 57.912 167.64 0)
+			(hide yes)
+			(show_name no)
+			(do_not_autoplace no)
+			(effects
+				(font
+					(size 1.27 1.27)
+				)
+				(justify bottom)
+			)
+		)
+		(property "Supplier Part Num" " 839-54-00274-ND"
+			(at 58.42 147.32 0)
+			(hide yes)
+			(show_name no)
+			(do_not_autoplace no)
+			(effects
+				(font
+					(size 1.27 1.27)
+				)
+			)
+		)
+		(pin "1"
+		)
+		(pin "S2"
+		)
+		(pin "4"
+		)
+		(pin "2"
+		)
+		(pin "S1"
+		)
+		(pin "3"
+		)
+		(instances
+			(project "dc-motor-driver"
+				(path "/fc286157-4263-4a46-ad05-98b3354aa28a"
+					(reference "J1")
+					(unit 1)
+				)
+			)
+		)
 	)
 	(symbol
@@
 					(unit 1)
 				)
-			)
-		)
-	)
-	(symbol
-		(lib_id "Manufacturer Connectors:54-00274")
-		(at 58.42 147.32 0)
-		(unit 1)
-		(body_style 1)
-		(exclude_from_sim no)
-		(in_bom yes)
-		(on_board yes)
-		(in_pos_files yes)
-		(dnp no)
-		(fields_autoplaced yes)
-		(property "Reference" "J14"
-			(at 59.055 134.62 0)
-			(show_name no)
-			(do_not_autoplace no)
-			(effects
-				(font
-					(size 1.27 1.27)
-				)
-			)
-		)
-		(property "Value" "54-00274"
-			(at 59.055 137.16 0)
-			(show_name no)
-			(do_not_autoplace no)
-			(effects
-				(font
-					(size 1.27 1.27)
-				)
-			)
-		)
-		(property "Footprint" "ConnectorsOther:Tensility_M8_Socket_4P_Shielded_A"
-			(at 58.42 147.32 0)
-			(hide yes)
-			(show_name no)
-			(do_not_autoplace no)
-			(effects
-				(font
-					(size 1.27 1.27)
-				)
-				(justify bottom)
-			)
-		)
-		(property "Datasheet" "https://tensility.s3.us-west-2.amazonaws.com/uploads/pdffiles/54-00274.pdf"
-			(at 58.42 147.32 0)
-			(hide yes)
-			(show_name no)
-			(do_not_autoplace no)
-			(effects
-				(font
-					(size 1.27 1.27)
-				)
-			)
-		)
-		(property "Description" ""
-			(at 58.42 147.32 0)
-			(hide yes)
-			(show_name no)
-			(do_not_autoplace no)
-			(effects
-				(font
-					(size 1.27 1.27)
-				)
-			)
-		)
-		(property "PARTREV" "A"
-			(at 58.42 147.32 0)
-			(hide yes)
-			(show_name no)
-			(do_not_autoplace no)
-			(effects
-				(font
-					(size 1.27 1.27)
-				)
-				(justify bottom)
-			)
-		)
-		(property "STANDARD" "Manufacturer Recommendations"
-			(at 58.42 147.32 0)
-			(hide yes)
-			(show_name no)
-			(do_not_autoplace no)
-			(effects
-				(font
-					(size 1.27 1.27)
-				)
-				(justify bottom)
-			)
-		)
-		(property "MAXIMUM_PACKAGE_HEIGHT" "13.54mm"
-			(at 58.42 147.32 0)
-			(hide yes)
-			(show_name no)
-			(do_not_autoplace no)
-			(effects
-				(font
-					(size 1.27 1.27)
-				)
-				(justify bottom)
-			)
-		)
-		(property "MANUFACTURER" "Tensility"
-			(at 58.42 147.32 0)
-			(hide yes)
-			(show_name no)
-			(do_not_autoplace no)
-			(effects
-				(font
-					(size 1.27 1.27)
-				)
-				(justify bottom)
-			)
-		)
-		(property "Supplier" "DigiKey"
-			(at 58.42 147.32 0)
-			(hide yes)
-			(show_name no)
-			(do_not_autoplace no)
-			(effects
-				(font
-					(size 1.27 1.27)
-				)
-			)
-		)
-		(property "Supplier Part No" " 839-54-00274-ND"
-			(at 58.42 147.32 0)
-			(hide yes)
-			(show_name no)
-			(do_not_autoplace no)
-			(effects
-				(font
-					(size 1.27 1.27)
-				)
-			)
-		)
-		(property "Supplier Link" "https://www.digikey.com.au/en/products/detail/tensility-international-corp/54-00274/16604946"
-			(at 58.42 147.32 0)
-			(hide yes)
-			(show_name no)
-			(do_not_autoplace no)
-			(effects
-				(font
-					(size 1.27 1.27)
-				)
-			)
-		)
-		(pin "S1"
-		)
-		(pin "2"
-		)
-		(pin "S2"
-		)
-		(pin "4"
-		)
-		(pin "3"
-		)
-		(pin "1"
-		)
-		(instances
-			(project "dc-motor-driver"
-				(path "/fc286157-4263-4a46-ad05-98b3354aa28a"
-					(reference "J14")
-					(unit 1)
-				)

Commit message: Fixed schematic element and bad symbol
Parts:
- J1: footprint ConnectorsOther:AnyTek_OQ_3.81mm_90_2P_TriangleKeyLock -> ConnectorsOther:Tensility_M8_Socket_4P_Shielded_A
Changed lines of the file:
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@@
 			)
 		)
-		(property "Footprint" "ConnectorsOther:AnyTek_OQ_3.81mm_90_2P_TriangleKeyLock"
+		(property "Footprint" "ConnectorsOther:Tensility_M8_Socket_4P_Shielded_A"
 			(at 82.042 160.274 0)
 			(hide yes)
