File: hardware/dc-motor-driver/dc-motor-driver.kicad_sch (KiCad schematic)
At the start: 20 parts, among them J2 VIN, J3 DE9, J4 Conn_01x02

Commit message: Prod ready, fixed silkscreen and chamfered, plus readjusted stat LED placement
Other:
- note added: "GPIO 39 and 38 can be used"
Changed lines of the file:
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@@
+		)
+	)
+	(text "GPIO 39 and 38 can be used"
+		(exclude_from_sim no)
+		(at 151.384 97.282 0)
+		(effects
+			(font
+				(size 1.27 1.27)
+			)
 		)
 	)
