Commit message: Fix RealSense D455 x-offset typo in sensor_mount
The D455 origin read xyz="10.035 0.0 0.006", placing the camera ten
metres in front of the mast. Correct to 0.035, matching the mast's
front face.

Co-Authored-By: Claude Opus 5 (1M context) <noreply@anthropic.com>

File: software/ros_ws/src/description/urdf/sensor_mount.urdf.xacro (robot description, xacro)
@@ -42,5 +42,5 @@
     <!-- RealSense D455, on the front face of the mast, looking straight ahead -->
     <xacro:sensor_d455 parent="${prefix}sensor_mount" name="camera" use_nominal_extrinsics="true">
-      <origin xyz="10.035 0.0 0.006" rpy="0.0 0.0 0.0"/>
+      <origin xyz="0.035 0.0 0.006" rpy="0.0 0.0 0.0"/>
     </xacro:sensor_d455>
     <xacro:camera_d455_gazebo name="camera"/>
