Commit message: Fix LiDAR pitch orientation and adjust RealSense D455 position for improved alignment

File: software/ros_ws/src/description/urdf/sensor_mount.urdf.xacro (robot description, xacro)
@@ -38,9 +38,9 @@
       <parent link="${prefix}sensor_mount"/>
       <child link="${prefix}livox_frame"/>
-      <origin xyz="0.04 0.0 0.13" rpy="0.0 ${livox_pitch} 0.0"/>
+      <origin xyz="0.04 0.0 0.13" rpy="${-livox_pitch} 0.0 ${0.0}"/>
     </joint>
     <!-- RealSense D455, on the front face of the mast, looking straight ahead -->
     <xacro:sensor_d455 parent="${prefix}sensor_mount" name="camera" use_nominal_extrinsics="true">
-      <origin xyz="0.035 0.0 0.006" rpy="0.0 0.0 0.0"/>
+      <origin xyz="10.035 0.0 0.006" rpy="0.0 0.0 0.0"/>
     </xacro:sensor_d455>
     <xacro:camera_d455_gazebo name="camera"/>

Commit message: Update sensor_mount.urdf.xacro to use correct mesh for LiDAR base
- Changed the mesh filename from 'sensor_mount.dae' to 'lidar_base.dae' for the LiDAR base link.
- Removed commented-out visual element to clean up the code.

File: software/ros_ws/src/description/urdf/sensor_mount.urdf.xacro (robot description, xacro)
@@ -36,13 +36,10 @@
     -->
     <link name="${prefix}livox_base">
-      <!-- no mesh for the plate yet: a visual without a geometry fails to parse, so the
-           whole element stays commented out until there is one to point at.
       <visual>
         <origin xyz="0.0 0.0 0.0" rpy="0.0 0.0 ${pi/2}"/>
         <geometry>
-          <mesh scale="1.0 1.0 1.0" filename="file://$(find description)/meshes/sensor_mount.dae"/>
+          <mesh scale="1.0 1.0 1.0" filename="file://$(find description)/meshes/lidar_base.dae"/>
         </geometry>
       </visual>
-      -->
     </link>
     <joint name="${prefix}livox_base_joint" type="fixed">

Commit message: Update livox_base and laser_joint origins in sensor_mount.urdf.xacro for improved alignment

File: software/ros_ws/src/description/urdf/sensor_mount.urdf.xacro (robot description, xacro)
@@ -37,5 +37,5 @@
     <link name="${prefix}livox_base">
       <visual>
-        <origin xyz="0.0 0.0 0.0" rpy="0.0 0.0 ${pi/2}"/>
+        <origin xyz="${-0.082} 0.0 ${0.002}" rpy="${pi/2} 0.0 ${pi}"/>
         <geometry>
           <mesh scale="1.0 1.0 1.0" filename="file://$(find description)/meshes/lidar_base.dae"/>
@@ -81,5 +81,5 @@
       <parent link="${prefix}livox_base"/>
       <child link="${prefix}livox_frame"/>
-      <origin xyz="${-0.08} 0.0 0.05" rpy="${0.0} 0.0 ${0.0}"/>
+      <origin xyz="${-0.038} 0.0 0.064" rpy="${0.0} 0.0 ${-pi/2}"/>
     </joint>
     <!-- RealSense D455, on the front face of the mast, looking straight ahead -->

Commit message: Stop laser_joint yawing the Livox frame 90 degrees
laser_joint carried rpy="0 0 -pi/2", added in 31015e3 "for improved
alignment", while the comment above it still said the joint "adds no
rotation of its own". The comment described the intent; the yaw was there
to line up the mesh.

It is not a cosmetic setting. base_link -> livox_frame resolved to
roll -45, pitch 0, yaw -90 rather than the intended pitch 45, and
fast_lio composes T_map_base = T_map_imu * T_imu_lidar * T_lidar_base
with lid_frame -> base_frame read straight from TF, so the yaw landed in
the pose it reports for base_link: base_link started 90 degrees off odom
the moment localisation came up. Gravity alignment cannot absorb that,
because an accelerometer constrains roll and pitch only, which is why
disabling common.gravity_align_en made no difference.

The -pi/2 moves into the visual and inertial origins, so the mesh renders
exactly as before, and the comment now says why the joint must stay
unrotated.

Verified by expanding perseus.urdf.xacro through xacro: base_link ->
livox_frame is now roll 0, pitch 45, yaw 0.

The same joint in perseus_simulation orients the Gazebo gpu_lidar and IMU,
which attach to livox_frame by reference with no pose of their own; it is
fixed there in its own commit.

File: software/ros_ws/src/description/urdf/sensor_mount.urdf.xacro (robot description, xacro)
@@ -55,10 +55,10 @@
     <link name="${prefix}livox_frame">
       <inertial>
-        <origin xyz="0 0.0 0.0" rpy="${pi/2} 0.0 ${pi}"/>
+        <origin xyz="0 0.0 0.0" rpy="${pi/2} 0.0 ${pi/2}"/>
         <mass value="${livox_mass}"/>
         <xacro:box_inertia m="${livox_mass}" x="${livox_length}" y="${livox_radius}" z="${livox_radius}"/>
       </inertial>
       <visual>
-        <origin xyz="0 0.0 -0.02" rpy="${pi/2} 0.0 ${pi}"/>
+        <origin xyz="0 0.0 -0.02" rpy="${pi/2} 0.0 ${pi/2}"/>
         <geometry>
           <mesh scale="1.0 1.0 1.0" filename="file://$(find description)/meshes/mid-360.dae"/>
@@ -77,9 +77,16 @@
       extrinsic in the fast_lio config is internal to the sensor housing and is unaffected
       by how the housing is mounted.
+      Do not add a rotation here to make the mesh line up. This joint is what says where the
+      sensor points, and fast_lio composes the robot's pose as
+      T_map_base = T_map_imu * T_imu_lidar * T_lidar_base, reading lid_frame -> base_frame
+      straight out of TF, so a yaw added here lands in base_link's reported orientation.
+      A -pi/2 put here for mesh alignment is exactly why base_link once started 90 degrees
+      off odom, and gravity alignment cannot absorb it, because an accelerometer constrains
+      roll and pitch only. Mesh alignment belongs on the <visual> origin above.
     -->
     <joint name="${prefix}laser_joint" type="fixed">
       <parent link="${prefix}livox_base"/>
       <child link="${prefix}livox_frame"/>
-      <origin xyz="${-0.038} 0.0 0.064" rpy="${0.0} 0.0 ${-pi/2}"/>
+      <origin xyz="${-0.038} 0.0 0.064" rpy="0.0 0.0 0.0"/>
     </joint>
     <!-- RealSense D455, on the front face of the mast, looking straight ahead -->

Commit message: restore the correct sensors orientation

File: software/ros_ws/src/description/urdf/sensor_mount.urdf.xacro (robot description, xacro)
@@ -55,10 +55,10 @@
     <link name="${prefix}livox_frame">
       <inertial>
-        <origin xyz="0 0.0 0.0" rpy="${pi/2} 0.0 ${pi/2}"/>
+        <origin xyz="0 0.0 0.0" rpy="${pi/2} 0.0 ${pi}"/>
         <mass value="${livox_mass}"/>
         <xacro:box_inertia m="${livox_mass}" x="${livox_length}" y="${livox_radius}" z="${livox_radius}"/>
       </inertial>
       <visual>
-        <origin xyz="0 0.0 -0.02" rpy="${pi/2} 0.0 ${pi/2}"/>
+        <origin xyz="0 0.0 -0.02" rpy="${pi/2} 0.0 ${pi}"/>
         <geometry>
           <mesh scale="1.0 1.0 1.0" filename="file://$(find description)/meshes/mid-360.dae"/>
@@ -77,16 +77,23 @@
       extrinsic in the fast_lio config is internal to the sensor housing and is unaffected
       by how the housing is mounted.
-      Do not add a rotation here to make the mesh line up. This joint is what says where the
-      sensor points, and fast_lio composes the robot's pose as
-      T_map_base = T_map_imu * T_imu_lidar * T_lidar_base, reading lid_frame -> base_frame
-      straight out of TF, so a yaw added here lands in base_link's reported orientation.
-      A -pi/2 put here for mesh alignment is exactly why base_link once started 90 degrees
-      off odom, and gravity alignment cannot absorb it, because an accelerometer constrains
-      roll and pitch only. Mesh alignment belongs on the <visual> origin above.
+      The -pi/2 yaw is not mesh alignment: the sensor is physically seated on the plate
+      rotated a quarter turn, so TF has to say so. livox_ros_driver2 stamps every cloud
+      frame_id: livox_frame, which means this joint's orientation is what orients every
+      point downstream; get it wrong and the whole point cloud is rotated.
+      96a84d2 removed this yaw (PR #17, fix/livox-frame-yaw) to stop base_link starting
+      90 degrees off odom, and that reversed the trade. fast_lio does compose
+      T_map_base = T_map_imu * T_imu_lidar * T_lidar_base with lid_frame -> base_frame read
+      from TF, so the yaw does land in base_link's reported orientation, but odom has no
+      absolute yaw reference (see the imu0 notes in autonomy_bringup/config/ekf_config.yaml),
+      so the odom frame is defined by wherever the robot started and a 90 degree offset in it
+      is cosmetic. A rotated point cloud is not. What has to agree is the cloud and the pose,
+      and only keeping the real mounting rotation here achieves that.
+      Mesh alignment is the pi on the <visual> and <inertial> origins above; the two move
+      together, so changing one without the other makes the model lie about the frame.
     -->
     <joint name="${prefix}laser_joint" type="fixed">
       <parent link="${prefix}livox_base"/>
       <child link="${prefix}livox_frame"/>
-      <origin xyz="${-0.038} 0.0 0.064" rpy="0.0 0.0 0.0"/>
+      <origin xyz="${-0.038} 0.0 0.064" rpy="${0.0} 0.0 ${-pi/2}"/>
     </joint>
     <!-- RealSense D455, on the front face of the mast, looking straight ahead -->

Commit message: feat: state the LiDAR-IMU extrinsic in the URDF, not in the LIO configs
The MID-360 datasheet offset between the LiDAR origin and the IMU inside the
housing was written out twice, as mapping.extrinsic_T in livox_mid360.yaml and
again as calibration.translation in bievr_mid360.yaml, with nothing checking the
two against each other. It is a physical property of the sensor, so it belongs in
the robot description next to laser_joint, and the LIO configs should be reading
it rather than restating it.

description gains livox_imu_frame, a pure frame under livox_frame at the
datasheet offset. No visual, no collision, no inertial: nothing about the robot's
mass or appearance depends on it, and Gazebo has no use for it either. Note the
sign, because it trips people up -- the joint states the IMU in LiDAR
coordinates, and both LIO configs express the extrinsic the other way round.

bievr_mid360.yaml now sets calibration.from_tf and drops the vectors, so
BIEVR-LIO reads the extrinsic as livox_imu_frame -> livox_frame at startup. That
makes the robot description a hard dependency of odometry, but it already was:
base.origin_at_base cannot place the world frame without it either, so nothing
new has to come up first. Bag replays have no live TF and need the vectors back.

livox_mid360.yaml keeps its copy, because FAST-LIO has no equivalent, but now
says where the authority is. A side effect worth having: common.body_frame there
has named livox_imu_frame all along, and until now that was a frame which did not
exist anywhere in the TF tree.

Pin moved to 0cd2b05.

Verified by expanding the real top-level description and confirming
livox_imu_joint comes out at (0.011, 0.02329, -0.04412) under livox_frame, then
running the nix-built node against a TF tree carrying that joint: it reports the
extrinsic it read as t = [-0.011, -0.02329, 0.04412] -- exactly what the config
used to hardcode -- and produces the same odometry, 1214 messages as odom ->
base_link with a stationary robot holding to 1 cm and 0.02 degrees. Not yet
tested on the robot or against Gazebo itself.

File: software/ros_ws/src/description/urdf/sensor_mount.urdf.xacro (robot description, xacro)
@@ -97,4 +97,26 @@
       <origin xyz="${-0.038} 0.0 0.064" rpy="${0.0} 0.0 ${-pi/2}"/>
     </joint>
+    <!--
+      The IMU inside the Livox housing. A pure frame: no visual, no collision, no inertial,
+      because nothing about the robot's mass or appearance depends on it and Gazebo has no
+      use for it either (the simulated IMU in sensors.urdf.xacro is attached to livox_frame,
+      which is 4.4 cm away, and that is irrelevant against a noise-free simulated sensor).
+      It exists so the LiDAR-IMU extrinsic has one home. The MID-360 datasheet puts the IMU
+      at (11.0, 23.29, -44.12) mm from the LiDAR origin, in LiDAR coordinates, with no
+      rotation between them. That number was previously written out twice, as
+      mapping.extrinsic_T in autonomy_bringup/config/livox_mid360.yaml and again as
+      calibration.translation in bievr_mid360.yaml, with nothing checking the two against
+      each other. Stating it here instead lets BIEVR-LIO read it back out of TF
+      (calibration.from_tf), and makes common.body_frame in the FAST-LIO config name a link
+      that actually exists.
+      Note the sign. Both LIO configs express the extrinsic the other way round, as the
+      LiDAR origin in IMU coordinates, so they carry the negation of these numbers.
+    -->
+    <link name="${prefix}livox_imu_frame"/>
+    <joint name="${prefix}livox_imu_joint" type="fixed">
+      <parent link="${prefix}livox_frame"/>
+      <child link="${prefix}livox_imu_frame"/>
+      <origin xyz="0.011 0.02329 ${-0.04412}" rpy="0.0 0.0 0.0"/>
+    </joint>
     <!-- RealSense D455, on the front face of the mast, looking straight ahead -->
     <xacro:sensor_d455 parent="${prefix}sensor_mount" name="camera" use_nominal_extrinsics="true">

Commit message: refactor(urdf): update mesh file paths to use package:// syntax for consistency

File: software/ros_ws/src/description/urdf/sensor_mount.urdf.xacro (robot description, xacro)
@@ -20,5 +20,5 @@
         <origin xyz="${-0.023} ${0.005} ${-0.035}" rpy="0.0 0.0 ${pi/2}"/>
         <geometry>
-          <mesh scale="1.0 1.0 1.0" filename="file://$(find description)/meshes/sensor_mount.dae"/>
+          <mesh scale="1.0 1.0 1.0" filename="package://description/meshes/sensor_mount.dae"/>
         </geometry>
       </visual>
@@ -39,5 +39,5 @@
         <origin xyz="${-0.082} 0.0 ${0.002}" rpy="${pi/2} 0.0 ${pi}"/>
         <geometry>
-          <mesh scale="1.0 1.0 1.0" filename="file://$(find description)/meshes/lidar_base.dae"/>
+          <mesh scale="1.0 1.0 1.0" filename="package://description/meshes/lidar_base.dae"/>
         </geometry>
       </visual>
@@ -62,5 +62,5 @@
         <origin xyz="0 0.0 -0.02" rpy="${pi/2} 0.0 ${pi}"/>
         <geometry>
-          <mesh scale="1.0 1.0 1.0" filename="file://$(find description)/meshes/mid-360.dae"/>
+          <mesh scale="1.0 1.0 1.0" filename="package://description/meshes/mid-360.dae"/>
         </geometry>
       </visual>
