Commit message: feat: Update mesh file paths to use package:// syntax for URDF files

File: software/ros_ws/src/description/urdf/chassis.urdf.xacro (robot description, xacro)
@@ -10,5 +10,5 @@
       <origin xyz="0.0 0.0 0.0" rpy="0 0.0 -${pi/2}"/>
       <geometry>
-        <mesh scale="0.1 0.1  0.1" filename="file://$(find description)/meshes/chassis.dae"/>
+        <mesh scale="0.1 0.1  0.1" filename="package://description/meshes/chassis.dae"/>
       </geometry>
     </visual>

File: software/ros_ws/src/description/urdf/flange_bearing.urdf.xacro (robot description, xacro)
@@ -11,5 +11,5 @@
     <origin xyz="0.0 0.0 0.0" rpy="${-pi/2} 0 ${pi/2}"/>
     <geometry>
-        <mesh scale="0.1 0.1  0.1" filename="file://$(find description)/meshes/flange_bearing.dae"/>
+        <mesh scale="0.1 0.1  0.1" filename="package://description/meshes/flange_bearing.dae"/>
     </geometry>
     </visual>
@@ -31,5 +31,5 @@
     <origin xyz="0.0 0.0 0.0" rpy="${-pi/2} 0 ${-pi/2}"/>
     <geometry>
-        <mesh scale=  "0.1 0.1  0.1" filename="file://$(find description)/meshes/differential_bar.dae"/>
+        <mesh scale=  "0.1 0.1  0.1" filename="package://description/meshes/differential_bar.dae"/>
     </geometry>
     </visual>

File: software/ros_ws/src/description/urdf/motor_wheel.urdf.xacro (robot description, xacro)
@@ -17,5 +17,5 @@
         </xacro:if>
         <geometry>
-          <mesh scale="0.1 0.1  0.1" filename="file://$(find description)/meshes/gearbox.dae"/>
+          <mesh scale="0.1 0.1  0.1" filename="package://description/meshes/gearbox.dae"/>
         </geometry>
         <!-- <material name="white"/> -->

File: software/ros_ws/src/description/urdf/rocker.urdf.xacro (robot description, xacro)
@@ -16,8 +16,8 @@
       <geometry>
       <xacro:if value="${side == 'left'}">
-        <mesh scale="0.1 0.1 0.1" filename="file://$(find description)/meshes/rocker_left.dae"/>
+        <mesh scale="0.1 0.1 0.1" filename="package://description/meshes/rocker_left.dae"/>
       </xacro:if>
       <xacro:if value="${side == 'right'}">
-        <mesh scale="0.1 0.1 0.1" filename="file://$(find description)/meshes/rocker_right.dae"/>
+        <mesh scale="0.1 0.1 0.1" filename="package://description/meshes/rocker_right.dae"/>
       </xacro:if>
       </geometry>

File: software/ros_ws/src/description/urdf/sensor_mount.urdf.xacro (robot description, xacro)
@@ -20,5 +20,5 @@
         <origin xyz="${-0.023} ${0.005} ${-0.035}" rpy="0.0 0.0 ${pi/2}"/>
         <geometry>
-          <mesh scale="1.0 1.0 1.0" filename="file://$(find description)/meshes/sensor_mount.dae"/>
+          <mesh scale="1.0 1.0 1.0" filename="package://description/meshes/sensor_mount.dae"/>
         </geometry>
       </visual>
@@ -39,5 +39,5 @@
         <origin xyz="${-0.082} 0.0 ${0.002}" rpy="${pi/2} 0.0 ${pi}"/>
         <geometry>
-          <mesh scale="1.0 1.0 1.0" filename="file://$(find description)/meshes/lidar_base.dae"/>
+          <mesh scale="1.0 1.0 1.0" filename="package://description/meshes/lidar_base.dae"/>
         </geometry>
       </visual>
@@ -62,5 +62,5 @@
         <origin xyz="0 0.0 -0.02" rpy="${pi/2} 0.0 ${pi}"/>
         <geometry>
-          <mesh scale="1.0 1.0 1.0" filename="file://$(find description)/meshes/mid-360.dae"/>
+          <mesh scale="1.0 1.0 1.0" filename="package://description/meshes/mid-360.dae"/>
         </geometry>
       </visual>

File: software/ros_ws/src/description/urdf/wheel.urdf.xacro (robot description, xacro)
@@ -18,5 +18,5 @@
       </xacro:if>
       <geometry>
-        <mesh scale="0.1 0.1 0.1" filename="file://$(find description)/meshes/wheel.dae"/>
+        <mesh scale="0.1 0.1 0.1" filename="package://description/meshes/wheel.dae"/>
       </geometry>
     </visual>
