Commit message: refactor: name the bucket meshes and frames like the rest of the description
The bucket linkage arrived with its Onshape export names, which look nothing
like the package around them. The 32 meshes were CAD assembly paths carrying
version and instance tokens - Bucket_1_Main_Bucket_Mount_Plate_v8_1_6mm_Bearing_v1_1.stl,
Left_Arm_-_Square_Tube_1.stl, and Acutator_on_Arm_Mount_1.stl with the CAD's own
misspelling - where every other mesh here is a flat lowercase part name like
chassis.dae or sensor_mount.dae. Separately, the five rams were the only bucket
frames not prefixed bucket_, so the assembly could not be found with one prefix.

Meshes are renamed after the part and the link that draws them, and converted
to COLLADA so the directory matches the other twelve meshes. assimp labels its
output Y_UP while leaving the vertices where they were, which would have rotated
every mesh a quarter turn on load, so each file is corrected to Z_UP - the same
coordinates-as-authored convention the existing meshes use, and what the STLs
were doing implicitly. Bounding boxes were compared before and after for all 32:
no change beyond float noise. They appear as delete-plus-add rather than renames
because the format changed.

Sides in the new names come from each visual's origin rather than the CAD
instance number, which is not trustworthy: the brackets are numbered 1, 2, 4,
the on-arm mounts 1 and 3, and both arm tubes are called "Left_Arm". So
Left_Arm_-_Square_Tube_1 sits at y +0.100 and becomes lift_arm_left, and _2 at
y -0.100 becomes lift_arm_right. The two Bucket_1_6mm_Bearing files are 24 mm
apart beside the v-slot mount rather than a left/right pair, so they are
numbered instead of given a side that would have been wrong.

The rams become bucket_ram_*, taking their ten joints with them, and the arm
becomes bucket_lift_arm to match the bucket_lift_arm_pivot_* frames already on
the mount. The bare bucket link becomes bucket_body, symmetric with bucket_jaw
and no longer ambiguous with the assembly. All 25 bucket links now share the
one prefix.

Left alone deliberately: bucket_lift_joint, bucket_tilt_joint and
bucket_jaw_joint, which are named for the motion to match bucket_driver's
LIFT_BOTH / TILT_BOTH / JAWS_BOTH groups and are the external interface; and the
/bucket/ram_*/cmd_* topics, which perseus_simulation's gz_bridge.yaml binds to
by name.

bucket_ram_follower.py moves in lockstep. This matters more than it looks: both
of its joint lookups sit in try/except blocks that simply return, and a missing
jaw joint is swallowed with q_jaw defaulted to zero, so a stale name would not
raise - the rams would just freeze and the jaw sit closed.

Verified in the dev profile: payload:=none still expands to 33 links, unchanged;
payload:=bucket gives 58 links and 61 joints; every mesh path resolves; the
viewer starts clean and the follower publishes all ten renamed ram joints, with
the sliders description marking them fixed so the panel still lists only the four
wheels plus lift, tilt and jaw.

Note for whoever reconciles the two repos: perseus_simulation's bucket-urdf
branch keeps the old vocabulary, so the descriptions no longer agree on names.

File: software/ros_ws/src/description/urdf/bucket_linkage.urdf.xacro (robot description, xacro)
@@ -189,5 +189,5 @@
       <visual>
         <origin xyz="${mesh_xyz}" rpy="${mesh_rpy}"/>
-        <geometry><mesh filename="${M}/${mesh}_base.stl"/></geometry>
+        <geometry><mesh scale="1.0 1.0 1.0" filename="${M}/${mesh}_barrel.dae"/></geometry>
         <material name="bucket_steel"/>
       </visual>
@@ -209,5 +209,5 @@
       <visual>
         <origin xyz="${mesh_xyz}" rpy="${mesh_rpy}"/>
-        <geometry><mesh filename="${M}/${mesh}_slider.stl"/></geometry>
+        <geometry><mesh scale="1.0 1.0 1.0" filename="${M}/${mesh}_shaft.dae"/></geometry>
         <material name="bucket_dark"/>
       </visual>
@@ -256,10 +256,10 @@
       <visual>
         <origin xyz="${barrel_xyz}" rpy="${barrel_rpy}"/>
-        <geometry><mesh filename="${M}/${base_mesh}.stl"/></geometry>
+        <geometry><mesh scale="1.0 1.0 1.0" filename="${M}/${base_mesh}.dae"/></geometry>
         <material name="bucket_dark"/>
       </visual>
     </link>
     <joint name="${prefix}${name}_pitch_joint" type="revolute">
-      <parent link="${prefix}bucket"/>
+      <parent link="${prefix}bucket_body"/>
       <child link="${prefix}${name}_barrel"/>
       <origin xyz="${jaw_ram_x} ${y} ${jaw_ram_z}" rpy="0 ${jaw_ram_phi0} 0"/>
@@ -276,5 +276,5 @@
       <visual>
         <origin xyz="${shaft_xyz}" rpy="${shaft_rpy}"/>
-        <geometry><mesh filename="${M}/${shaft_mesh}.stl"/></geometry>
+        <geometry><mesh scale="1.0 1.0 1.0" filename="${M}/${shaft_mesh}.dae"/></geometry>
         <material name="bucket_steel"/>
       </visual>
@@ -333,5 +333,5 @@
          faithfully here.
          ═══════════════════════════════════════════════════════════════════ -->
-    <link name="${prefix}bucket_arm">
+    <link name="${prefix}bucket_lift_arm">
       <inertial>
         <origin xyz="0.407179 0.019695 -0.000497" rpy="0 0 0"/>
@@ -343,43 +343,43 @@
       <visual>
         <origin xyz="0.00004  0.10000 -0.00001" rpy="1.5707963 0 0"/>
-        <geometry><mesh filename="${M}/Left_Arm_-_Square_Tube_1.stl"/></geometry>
+        <geometry><mesh scale="1.0 1.0 1.0" filename="${M}/lift_arm_left.dae"/></geometry>
         <material name="bucket_arm_blue"/>
       </visual>
       <visual>
         <origin xyz="0.00004 -0.10000 -0.00001" rpy="1.5707963 0 0"/>
-        <geometry><mesh filename="${M}/Left_Arm_-_Square_Tube_2.stl"/></geometry>
+        <geometry><mesh scale="1.0 1.0 1.0" filename="${M}/lift_arm_right.dae"/></geometry>
         <material name="bucket_arm_blue"/>
       </visual>
       <visual>
         <origin xyz="0.59704 -0.08000 -0.01001" rpy="0 0 -1.5707963"/>
-        <geometry><mesh filename="${M}/Actuator_Bracket_1.stl"/></geometry>
+        <geometry><mesh scale="1.0 1.0 1.0" filename="${M}/lift_ram_bracket_right.dae"/></geometry>
         <material name="bucket_dark"/>
       </visual>
       <visual>
         <origin xyz="0.59704  0.12000 -0.01001" rpy="0 0 -1.5707963"/>
-        <geometry><mesh filename="${M}/Actuator_Bracket_2.stl"/></geometry>
+        <geometry><mesh scale="1.0 1.0 1.0" filename="${M}/lift_ram_bracket_left.dae"/></geometry>
         <material name="bucket_dark"/>
       </visual>
       <visual>
         <origin xyz="0.22674 -0.08000  0.00999" rpy="3.1415927 0 0"/>
-        <geometry><mesh filename="${M}/Acutator_on_Arm_Mount_1.stl"/></geometry>
+        <geometry><mesh scale="1.0 1.0 1.0" filename="${M}/tilt_ram_mount_outboard.dae"/></geometry>
         <material name="bucket_steel"/>
       </visual>
       <visual>
         <origin xyz="0.17904 -0.08000  0.01199" rpy="0 0 0"/>
-        <geometry><mesh filename="${M}/Acutator_on_Arm_Mount_3.stl"/></geometry>
+        <geometry><mesh scale="1.0 1.0 1.0" filename="${M}/tilt_ram_mount_inboard.dae"/></geometry>
         <material name="bucket_steel"/>
       </visual>
       <visual>
         <origin xyz="0.18674  0.02000  0.01399" rpy="-3.1415927 0 -1.5707963"/>
-        <geometry><mesh filename="${M}/Actuator_Bracket_4.stl"/></geometry>
+        <geometry><mesh scale="1.0 1.0 1.0" filename="${M}/tilt_ram_bracket.dae"/></geometry>
         <material name="bucket_dark"/>
       </visual>
       <!-- one box per tube, sized from the measured 750 x 40 x 20 extents -->
-      <collision name="${prefix}bucket_arm_left_collision">
+      <collision name="${prefix}bucket_lift_arm_left_collision">
         <origin xyz="0.35200 0.12000 0.00000" rpy="0 0 0"/>
         <geometry><box size="0.750 0.040 0.020"/></geometry>
       </collision>
-      <collision name="${prefix}bucket_arm_right_collision">
+      <collision name="${prefix}bucket_lift_arm_right_collision">
         <origin xyz="0.35200 -0.08000 0.00000" rpy="0 0 0"/>
         <geometry><box size="0.750 0.040 0.020"/></geometry>
@@ -390,5 +390,5 @@
     <joint name="${prefix}bucket_lift_joint" type="revolute">
       <parent link="${prefix}bucket_frame"/>
-      <child link="${prefix}bucket_arm"/>
+      <child link="${prefix}bucket_lift_arm"/>
       <origin xyz="0 0 0" rpy="0 ${lift_zero_pitch} 0"/>
       <axis xyz="0 -1 0"/>
@@ -411,5 +411,5 @@
          z -0.050..0.171.
          ═══════════════════════════════════════════════════════════════════ -->
-    <link name="${prefix}bucket">
+    <link name="${prefix}bucket_body">
       <inertial>
         <origin xyz="0.021877 0.111881 0.038577" rpy="0 0 0"/>
@@ -421,75 +421,75 @@
       <visual>
         <origin xyz="0.000003 -0.000002 -0.000004" rpy="0.0000000 -1.5707963 -1.5707963"/>
-        <geometry><mesh filename="${M}/Bucket_1_Main_Bucket_Mount_Plate_v8_1_Main_Bearing_Block_1.stl"/></geometry>
+        <geometry><mesh scale="1.0 1.0 1.0" filename="${M}/tilt_bearing_block_right.dae"/></geometry>
         <material name="bucket_dark"/>
       </visual>
       <visual>
         <origin xyz="0.041739 -0.024002 -0.020065" rpy="-1.5707964 -0.0000000 -1.5707963"/>
-        <geometry><mesh filename="${M}/Bucket_1_Bucket_REAR_Frame_1.stl"/></geometry>
+        <geometry><mesh scale="1.0 1.0 1.0" filename="${M}/bucket_body.dae"/></geometry>
         <material name="bucket_steel"/>
       </visual>
       <visual>
         <origin xyz="0.000003 -0.003002 -0.000004" rpy="0.0000000 -1.5707963 1.5707964"/>
-        <geometry><mesh filename="${M}/Bucket_1_Main_Bucket_Mount_Plate_v8_1_6mm_Bearing_v1_1.stl"/></geometry>
+        <geometry><mesh scale="1.0 1.0 1.0" filename="${M}/tilt_bearing_right_1.dae"/></geometry>
         <material name="bucket_dark"/>
       </visual>
       <visual>
         <origin xyz="0.000003 0.046998 -0.000004" rpy="0.0000000 -1.5707963 -1.5707963"/>
-        <geometry><mesh filename="${M}/Bucket_1_Main_Bucket_Mount_Plate_v8_1_6mm_Bearing_v1_4.stl"/></geometry>
+        <geometry><mesh scale="1.0 1.0 1.0" filename="${M}/tilt_bearing_right_4.dae"/></geometry>
         <material name="bucket_dark"/>
       </visual>
       <visual>
         <origin xyz="0.041739 0.138498 0.086935" rpy="-1.5707964 -0.0000000 -1.5707963"/>
-        <geometry><mesh filename="${M}/Bucket_1_BucketClipVslotMount_1.stl"/></geometry>
+        <geometry><mesh scale="1.0 1.0 1.0" filename="${M}/bucket_vslot_mount.dae"/></geometry>
         <material name="bucket_steel"/>
       </visual>
       <visual>
         <origin xyz="0.041739 0.175998 -0.020065" rpy="-1.5707964 -0.0000000 -1.5707963"/>
-        <geometry><mesh filename="${M}/Bucket_1_Main_Bucket_Mount_Plate_v8_2_Main_Bearing_Block_1.stl"/></geometry>
+        <geometry><mesh scale="1.0 1.0 1.0" filename="${M}/tilt_bearing_block_left.dae"/></geometry>
         <material name="bucket_dark"/>
       </visual>
       <visual>
         <origin xyz="0.000003 -0.009002 -0.000004" rpy="0.0000000 -1.5707963 1.5707964"/>
-        <geometry><mesh filename="${M}/Bucket_1_Main_Bucket_Mount_Plate_v8_1_6mm_Bearing_v1_2.stl"/></geometry>
+        <geometry><mesh scale="1.0 1.0 1.0" filename="${M}/tilt_bearing_right_2.dae"/></geometry>
         <material name="bucket_dark"/>
       </visual>
       <visual>
         <origin xyz="0.000003 0.052998 -0.000004" rpy="0.0000000 -1.5707963 -1.5707963"/>
-        <geometry><mesh filename="${M}/Bucket_1_Main_Bucket_Mount_Plate_v8_1_6mm_Bearing_v1_3.stl"/></geometry>
+        <geometry><mesh scale="1.0 1.0 1.0" filename="${M}/tilt_bearing_right_3.dae"/></geometry>
         <material name="bucket_dark"/>
       </visual>
       <visual>
         <origin xyz="0.044413 0.109998 0.123301" rpy="-1.5707963 -0.0000000 -3.1415926"/>
-        <geometry><mesh filename="${M}/Bucket_1_6mm_Bearing_v1_1.stl"/></geometry>
+        <geometry><mesh scale="1.0 1.0 1.0" filename="${M}/bucket_vslot_bearing_1.dae"/></geometry>
         <material name="bucket_dark"/>
       </visual>
       <visual>
         <origin xyz="0.044413 0.133998 0.123301" rpy="1.5707964 -0.0000000 -3.1415926"/>
-        <geometry><mesh filename="${M}/Bucket_1_6mm_Bearing_v1_2.stl"/></geometry>
+        <geometry><mesh scale="1.0 1.0 1.0" filename="${M}/bucket_vslot_bearing_2.dae"/></geometry>
         <material name="bucket_dark"/>
       </visual>
       <visual>
         <origin xyz="0.046739 0.175998 -0.020065" rpy="0.0000000 1.5707963 0.0000000"/>
-        <geometry><mesh filename="${M}/Bucket_1_Main_Bucket_Mount_Plate_v8_2_6mm_Bearing_v1_1.stl"/></geometry>
+        <geometry><mesh scale="1.0 1.0 1.0" filename="${M}/tilt_bearing_left_1.dae"/></geometry>
         <material name="bucket_dark"/>
       </visual>
       <visual>
         <origin xyz="-0.003261 0.175998 -0.020065" rpy="0.0000000 1.5707963 -3.1415927"/>
-        <geometry><mesh filename="${M}/Bucket_1_Main_Bucket_Mount_Plate_v8_2_6mm_Bearing_v1_4.stl"/></geometry>
+        <geometry><mesh scale="1.0 1.0 1.0" filename="${M}/tilt_bearing_left_4.dae"/></geometry>
         <material name="bucket_dark"/>
       </visual>
       <visual>
         <origin xyz="0.052739 0.175998 -0.020065" rpy="0.0000000 1.5707963 0.0000000"/>
-        <geometry><mesh filename="${M}/Bucket_1_Main_Bucket_Mount_Plate_v8_2_6mm_Bearing_v1_2.stl"/></geometry>
+        <geometry><mesh scale="1.0 1.0 1.0" filename="${M}/tilt_bearing_left_2.dae"/></geometry>
         <material name="bucket_dark"/>
       </visual>
       <visual>
         <origin xyz="-0.009261 0.175998 -0.020065" rpy="0.0000000 1.5707963 -3.1415927"/>
-        <geometry><mesh filename="${M}/Bucket_1_Main_Bucket_Mount_Plate_v8_2_6mm_Bearing_v1_3.stl"/></geometry>
+        <geometry><mesh scale="1.0 1.0 1.0" filename="${M}/tilt_bearing_left_3.dae"/></geometry>
         <material name="bucket_dark"/>
       </visual>
       <!-- The back plate, as a box. The tray and side structures are on the jaw
            link below, because they swing with it. -->
-      <collision name="${prefix}bucket_rear_collision">
+      <collision name="${prefix}bucket_body_collision">
         <origin xyz="0.04500 0.12200 0.03300" rpy="0 0 0"/>
         <geometry><box size="0.010 0.460 0.145"/></geometry>
@@ -499,6 +499,6 @@
          Zero is the CAD pose. -->
     <joint name="${prefix}bucket_tilt_joint" type="revolute">
-      <parent link="${prefix}bucket_arm"/>
-      <child link="${prefix}bucket"/>
+      <parent link="${prefix}bucket_lift_arm"/>
+      <child link="${prefix}bucket_body"/>
       <origin xyz="${arm_length} ${bucket_pivot_y} -0.00001" rpy="0 0 0"/>
       <axis xyz="0 -1 0"/>
@@ -519,5 +519,5 @@
          ═══════════════════════════════════════════════════════════════════ -->
     <joint name="${prefix}bucket_jaw_joint" type="revolute">
-      <parent link="${prefix}bucket"/>
+      <parent link="${prefix}bucket_body"/>
       <child link="${prefix}bucket_jaw"/>
       <origin xyz="0.076453 0.348498 0.158935" rpy="0 0 0"/>
@@ -537,5 +537,5 @@
       <visual>
         <origin xyz="0.000000 0.000000 0.000000" rpy="1.5707963 0.0000000 0.0000000"/>
-        <geometry><mesh filename="${M}/Bucket_1_Bucket_FRONT_Frame_1.stl"/></geometry>
+        <geometry><mesh scale="1.0 1.0 1.0" filename="${M}/bucket_jaw.dae"/></geometry>
         <material name="bucket_steel"/>
       </visual>
@@ -569,12 +569,12 @@
          block rather than showing as a gap at the visible rod end. Verified
          over the whole workspace: rod end lands within 0.01 mm. -->
-    <xacro:bucket_ram name="ram_lift_left"  parent="bucket_frame" mesh="250mm_Actuator_1"
+    <xacro:bucket_ram name="bucket_ram_lift_left"  parent="bucket_frame" mesh="lift_ram_left"
                       xyz="0.00004 0.119074 -0.24001"
                       mesh_rpy="0 -1.5707963 -1.5707963" axis="1 0 0" phi="0"/>
-    <xacro:bucket_ram name="ram_lift_right" parent="bucket_frame" mesh="250mm_Actuator_2"
+    <xacro:bucket_ram name="bucket_ram_lift_right" parent="bucket_frame" mesh="lift_ram_right"
                       xyz="0.00004 -0.079074 -0.24001"
                       mesh_rpy="0 -1.5707963 1.5707963" axis="1 0 0" phi="0"/>
     <!-- The tilt ram's barrel is bolted to the plate on the ARMS (the
-         Acutator_on_Arm_Mount pair, via Actuator_Bracket_4) and its rod reaches
+         tilt_ram_mount pair, via tilt_ram_bracket) and its rod reaches
          forward to the bucket. The CAD export describes it the other way round
          - Revolute_9's parent is Bucket_1 - because the toolkit roots each mate
@@ -584,17 +584,17 @@
          mesh_xyz places the actuator mesh so its arm-side pin sits on the joint
          rather than its origin. -->
-    <xacro:bucket_ram name="ram_tilt" parent="bucket_arm" mesh="250mm_Actuator_3"
+    <xacro:bucket_ram name="bucket_ram_tilt" parent="bucket_lift_arm" mesh="tilt_ram"
                       xyz="0.18674 0.030248 0.01399"
                       mesh_xyz="0.365 -0.02025 0"
                       mesh_rpy="0 1.5707963 -1.5707963" axis="1 0 0" phi="0"/>
     <!-- The two 50 mm jaw actuators. Right side is -y (act 1), left is +y (act 2). -->
-    <xacro:bucket_jaw_ram name="ram_jaw_right" y="-0.08137"
-        base_mesh="Bucket_1_50mm_Actuator_v4_1_1_Base_Actuator_v2_1"
-        shaft_mesh="Bucket_1_50mm_Actuator_v4_1_1_Shaft_v2_1"
+    <xacro:bucket_jaw_ram name="bucket_ram_jaw_right" y="-0.08137"
+        base_mesh="jaw_ram_right_barrel"
+        shaft_mesh="jaw_ram_right_shaft"
         barrel_xyz="0 0.02287 0" barrel_rpy="0 1.5707963 -1.5707963"
         shaft_xyz="0.20681 -0.02013 0" shaft_rpy="0 1.5707963 1.5707963"/>
-    <xacro:bucket_jaw_ram name="ram_jaw_left" y="0.32537"
-        base_mesh="Bucket_1_50mm_Actuator_v4_1_2_Base_Actuator_v2_1"
-        shaft_mesh="Bucket_1_50mm_Actuator_v4_1_2_Shaft_v2_1"
+    <xacro:bucket_jaw_ram name="bucket_ram_jaw_left" y="0.32537"
+        base_mesh="jaw_ram_left_barrel"
+        shaft_mesh="jaw_ram_left_shaft"
         barrel_xyz="0 0.0092 0" barrel_rpy="0 1.5707963 1.5707963"
         shaft_xyz="0.20681 0.02013 0" shaft_rpy="0 1.5707963 -1.5707963"/>
@@ -608,8 +608,8 @@
     <xacro:bucket_encoder name="bucket_lift_encoder_left"  parent="bucket_frame" xyz="0 0.1 0"/>
     <xacro:bucket_encoder name="bucket_lift_encoder_right" parent="bucket_frame" xyz="0 -0.1 0"/>
-    <xacro:bucket_encoder name="bucket_tilt_encoder_left"  parent="bucket_arm"   xyz="${arm_length} 0.100 -0.00001"/>
-    <xacro:bucket_encoder name="bucket_tilt_encoder_right" parent="bucket_arm"   xyz="${arm_length} ${bucket_pivot_y} -0.00001"/>
-    <xacro:bucket_encoder name="bucket_jaw_encoder_left"   parent="bucket"       xyz="0.076453 0.348498 0.158935"/>
-    <xacro:bucket_encoder name="bucket_jaw_encoder_right"  parent="bucket"       xyz="0.076453 -0.104502 0.158935"/>
+    <xacro:bucket_encoder name="bucket_tilt_encoder_left"  parent="bucket_lift_arm"   xyz="${arm_length} 0.100 -0.00001"/>
+    <xacro:bucket_encoder name="bucket_tilt_encoder_right" parent="bucket_lift_arm"   xyz="${arm_length} ${bucket_pivot_y} -0.00001"/>
+    <xacro:bucket_encoder name="bucket_jaw_encoder_left"   parent="bucket_body"       xyz="0.076453 0.348498 0.158935"/>
+    <xacro:bucket_encoder name="bucket_jaw_encoder_right"  parent="bucket_body"       xyz="0.076453 -0.104502 0.158935"/>
   </xacro:macro>
 </robot>
