Commit message: refactor: put the bucket's structural frames on the machine centre line
bucket_mount sits on the centre line but nothing below it did. bucket_frame and
bucket_lift_arm were 20 mm to one side, bucket_body 122 mm, and bucket_jaw
226 mm - so a frame's y told you where the CAD happened to put an origin rather
than how far off centre the part actually is, and reading the tree meant
carrying those offsets in your head.

The parts themselves were never off centre. lift_arm_left and lift_arm_right
sit at +-0.1000, bucket_body.dae and bucket_jaw.dae at 0.0000, the jaw rams at
+-0.2034: the geometry is symmetric and always was. Only the frames carrying it
were offset, which the inertials confirm independently - the frame's centre of
mass was at y +0.019998 and the arm's at +0.019695, both landing on zero once
the 20 mm comes out.

So each of the four frames moves onto the centre line and the offset it was
carrying moves into the origins inside that link: its inertial, its visuals and
collisions, and the joints to its children. bucket_pivot_y is gone, its 0.102 m
now expressed where it belongs, in bucket_body's own origins; the fact it
documented, that the bucket hangs off one arm rather than between both, is
restated at the tilt joint.

This is safe to do because lift, tilt and jaw all turn about y and the shifts are
along y. A revolute axis is the line through the joint origin, so sliding the
origin along that same line leaves the axis exactly where it was - the
compensation is therefore exact at every joint angle, not just at rest.

Verified by transforming every visual and collision into world coordinates
before and after, meshes included: 70 entries, worst displacement 0.000000 mm at
rest, and 0.000000 mm again at lift -0.55, tilt +0.90, jaw -0.40 rad. The link
count is unchanged at 58, the viewer starts clean and the follower still
publishes all ten ram joints.

Falling out of this, the pairs now read as pairs: the lift rams are +-0.099074
and the jaw rams +-0.20337 in their parent frames, where before they were
0.119074/-0.079074 and 0.32537/-0.08137.

Left as they are, because changing them would move hardware rather than
relabel it: the lift encoders remain at +0.080/-0.120 and the tilt encoders at
+0.080/-0.122. Both are genuinely asymmetric in the model. The lift pair in
particular should probably sit on the lift axis at +-0.100, where the pivot
frames put it, so that is worth a look - but it is a geometry fix, not this.

File: software/ros_ws/src/description/urdf/bucket_linkage.urdf.xacro (robot description, xacro)
@@ -24,8 +24,15 @@
        front face (frame-mesh coordinates: face centre (0.0174, 0.4607, 0.093), pivot
        midpoint (0.0591, 0.44071, 0.213)). x and z agree with the +0.042 / +-0.12 that
-       bucket.urdf.xacro puts its lift pivot frames at. y is -0.020, not 0: in the CAD
-       the arm pivots sit at -0.12 and +0.08 from the face centre, not symmetrically. -->
+       bucket.urdf.xacro puts its lift pivot frames at.
+       y is 0: bucket_frame, bucket_lift_arm, bucket_body and bucket_jaw all sit on the
+       machine centre line, like bucket_mount, so a frame's y tells you how far off
+       centre a part is rather than where the CAD happened to put its origin. The CAD is
+       offset - its arm pivots are at -0.12 and +0.08 from the face centre, and the
+       bucket hangs off one arm - and that offset now lives in the child origins inside
+       each link instead of in the frame itself. Nothing moves: lift, tilt and jaw all
+       turn about y, so sliding a frame along y leaves its axis line exactly where it
+       was, at any joint angle. -->
   <xacro:property name="bucket_frame_x" value="0.0417"/>
-  <xacro:property name="bucket_frame_y" value="-0.020"/>
+  <xacro:property name="bucket_frame_y" value="0.0"/>
   <xacro:property name="bucket_frame_z" value="0.120"/>
   <!-- ══ Density ═════════════════════════════════════════════════════════
@@ -50,7 +57,4 @@
   <!-- arm pivot -> bucket pivot, along the arm -->
   <xacro:property name="arm_length" value="0.70004"/>
-  <!-- lateral offset from the arm-pivot midpoint to the bucket pivot: the
-       bucket hangs off ONE arm (Revolute_2 on Square_Tube_2), not both -->
-  <xacro:property name="bucket_pivot_y" value="-0.10200"/>
   <!-- arm pivot -> lift-actuator bracket, along the arm (Fastened_2) -->
   <xacro:property name="lift_rod_offset" value="0.59712"/>
@@ -312,5 +316,5 @@
     <link name="${prefix}bucket_frame">
       <inertial>
-        <origin xyz="-0.033899 0.019998 -0.155044" rpy="0 0 0"/>
+        <origin xyz="-0.033899 -0.000002 -0.155044" rpy="0 0 0"/>
         <mass value="${4.2099*k}"/>
         <inertia ixx="${0.114994*k}" ixy="${0.0*k}"      ixz="${0.001957*k}"
@@ -335,5 +339,5 @@
     <link name="${prefix}bucket_lift_arm">
       <inertial>
-        <origin xyz="0.407179 0.019695 -0.000497" rpy="0 0 0"/>
+        <origin xyz="0.407179 -0.000305 -0.000497" rpy="0 0 0"/>
         <mass value="${2.8599*k}"/>
         <inertia ixx="${0.022280*k}" ixy="${0.000424*k}" ixz="${0.004437*k}"
@@ -342,35 +346,35 @@
       </inertial>
       <visual>
-        <origin xyz="0.00004  0.10000 -0.00001" rpy="1.5707963 0 0"/>
+        <origin xyz="0.00004 0.08 -0.00001" rpy="1.5707963 0 0"/>
         <geometry><mesh scale="1.0 1.0 1.0" filename="${M}/lift_arm_left.dae"/></geometry>
         <material name="bucket_arm_blue"/>
       </visual>
       <visual>
-        <origin xyz="0.00004 -0.10000 -0.00001" rpy="1.5707963 0 0"/>
+        <origin xyz="0.00004 -0.12 -0.00001" rpy="1.5707963 0 0"/>
         <geometry><mesh scale="1.0 1.0 1.0" filename="${M}/lift_arm_right.dae"/></geometry>
         <material name="bucket_arm_blue"/>
       </visual>
       <visual>
-        <origin xyz="0.59704 -0.08000 -0.01001" rpy="0 0 -1.5707963"/>
+        <origin xyz="0.59704 -0.1 -0.01001" rpy="0 0 -1.5707963"/>
         <geometry><mesh scale="1.0 1.0 1.0" filename="${M}/lift_ram_bracket_right.dae"/></geometry>
         <material name="bucket_dark"/>
       </visual>
       <visual>
-        <origin xyz="0.59704  0.12000 -0.01001" rpy="0 0 -1.5707963"/>
+        <origin xyz="0.59704 0.1 -0.01001" rpy="0 0 -1.5707963"/>
         <geometry><mesh scale="1.0 1.0 1.0" filename="${M}/lift_ram_bracket_left.dae"/></geometry>
         <material name="bucket_dark"/>
       </visual>
       <visual>
-        <origin xyz="0.22674 -0.08000  0.00999" rpy="3.1415927 0 0"/>
+        <origin xyz="0.22674 -0.1 0.00999" rpy="3.1415927 0 0"/>
         <geometry><mesh scale="1.0 1.0 1.0" filename="${M}/tilt_ram_mount_outboard.dae"/></geometry>
         <material name="bucket_steel"/>
       </visual>
       <visual>
-        <origin xyz="0.17904 -0.08000  0.01199" rpy="0 0 0"/>
+        <origin xyz="0.17904 -0.1 0.01199" rpy="0 0 0"/>
         <geometry><mesh scale="1.0 1.0 1.0" filename="${M}/tilt_ram_mount_inboard.dae"/></geometry>
         <material name="bucket_steel"/>
       </visual>
       <visual>
-        <origin xyz="0.18674  0.02000  0.01399" rpy="-3.1415927 0 -1.5707963"/>
+        <origin xyz="0.18674 0 0.01399" rpy="-3.1415927 0 -1.5707963"/>
         <geometry><mesh scale="1.0 1.0 1.0" filename="${M}/tilt_ram_bracket.dae"/></geometry>
         <material name="bucket_dark"/>
@@ -378,9 +382,9 @@
       <!-- one box per tube, sized from the measured 750 x 40 x 20 extents -->
       <collision name="${prefix}bucket_lift_arm_left_collision">
-        <origin xyz="0.35200 0.12000 0.00000" rpy="0 0 0"/>
+        <origin xyz="0.35200 0.1 0.00000" rpy="0 0 0"/>
         <geometry><box size="0.750 0.040 0.020"/></geometry>
       </collision>
       <collision name="${prefix}bucket_lift_arm_right_collision">
-        <origin xyz="0.35200 -0.08000 0.00000" rpy="0 0 0"/>
+        <origin xyz="0.35200 -0.1 0.00000" rpy="0 0 0"/>
         <geometry><box size="0.750 0.040 0.020"/></geometry>
       </collision>
@@ -413,5 +417,5 @@
     <link name="${prefix}bucket_body">
       <inertial>
-        <origin xyz="0.021877 0.111881 0.038577" rpy="0 0 0"/>
+        <origin xyz="0.021877 -0.010119 0.038577" rpy="0 0 0"/>
         <mass value="${3.3886*k}"/>
         <inertia ixx="${0.079246*k}" ixy="${0.000096*k}" ixz="${-0.001948*k}"
@@ -420,70 +424,70 @@
       </inertial>
       <visual>
-        <origin xyz="0.000003 -0.000002 -0.000004" rpy="0.0000000 -1.5707963 -1.5707963"/>
+        <origin xyz="0.000003 -0.122002 -0.000004" rpy="0.0000000 -1.5707963 -1.5707963"/>
         <geometry><mesh scale="1.0 1.0 1.0" filename="${M}/tilt_bearing_block_right.dae"/></geometry>
         <material name="bucket_dark"/>
       </visual>
       <visual>
-        <origin xyz="0.041739 -0.024002 -0.020065" rpy="-1.5707964 -0.0000000 -1.5707963"/>
+        <origin xyz="0.041739 -0.146002 -0.020065" rpy="-1.5707964 -0.0000000 -1.5707963"/>
         <geometry><mesh scale="1.0 1.0 1.0" filename="${M}/bucket_body.dae"/></geometry>
         <material name="bucket_steel"/>
       </visual>
       <visual>
-        <origin xyz="0.000003 -0.003002 -0.000004" rpy="0.0000000 -1.5707963 1.5707964"/>
+        <origin xyz="0.000003 -0.125002 -0.000004" rpy="0.0000000 -1.5707963 1.5707964"/>
         <geometry><mesh scale="1.0 1.0 1.0" filename="${M}/tilt_bearing_right_1.dae"/></geometry>
         <material name="bucket_dark"/>
       </visual>
       <visual>
-        <origin xyz="0.000003 0.046998 -0.000004" rpy="0.0000000 -1.5707963 -1.5707963"/>
+        <origin xyz="0.000003 -0.075002 -0.000004" rpy="0.0000000 -1.5707963 -1.5707963"/>
         <geometry><mesh scale="1.0 1.0 1.0" filename="${M}/tilt_bearing_right_4.dae"/></geometry>
         <material name="bucket_dark"/>
       </visual>
       <visual>
-        <origin xyz="0.041739 0.138498 0.086935" rpy="-1.5707964 -0.0000000 -1.5707963"/>
+        <origin xyz="0.041739 0.016498 0.086935" rpy="-1.5707964 -0.0000000 -1.5707963"/>
         <geometry><mesh scale="1.0 1.0 1.0" filename="${M}/bucket_vslot_mount.dae"/></geometry>
         <material name="bucket_steel"/>
       </visual>
       <visual>
-        <origin xyz="0.041739 0.175998 -0.020065" rpy="-1.5707964 -0.0000000 -1.5707963"/>
+        <origin xyz="0.041739 0.053998 -0.020065" rpy="-1.5707964 -0.0000000 -1.5707963"/>
         <geometry><mesh scale="1.0 1.0 1.0" filename="${M}/tilt_bearing_block_left.dae"/></geometry>
         <material name="bucket_dark"/>
       </visual>
       <visual>
-        <origin xyz="0.000003 -0.009002 -0.000004" rpy="0.0000000 -1.5707963 1.5707964"/>
+        <origin xyz="0.000003 -0.131002 -0.000004" rpy="0.0000000 -1.5707963 1.5707964"/>
         <geometry><mesh scale="1.0 1.0 1.0" filename="${M}/tilt_bearing_right_2.dae"/></geometry>
         <material name="bucket_dark"/>
       </visual>
       <visual>
-        <origin xyz="0.000003 0.052998 -0.000004" rpy="0.0000000 -1.5707963 -1.5707963"/>
+        <origin xyz="0.000003 -0.069002 -0.000004" rpy="0.0000000 -1.5707963 -1.5707963"/>
         <geometry><mesh scale="1.0 1.0 1.0" filename="${M}/tilt_bearing_right_3.dae"/></geometry>
         <material name="bucket_dark"/>
       </visual>
       <visual>
-        <origin xyz="0.044413 0.109998 0.123301" rpy="-1.5707963 -0.0000000 -3.1415926"/>
+        <origin xyz="0.044413 -0.012002 0.123301" rpy="-1.5707963 -0.0000000 -3.1415926"/>
         <geometry><mesh scale="1.0 1.0 1.0" filename="${M}/bucket_vslot_bearing_1.dae"/></geometry>
         <material name="bucket_dark"/>
       </visual>
       <visual>
-        <origin xyz="0.044413 0.133998 0.123301" rpy="1.5707964 -0.0000000 -3.1415926"/>
+        <origin xyz="0.044413 0.011998 0.123301" rpy="1.5707964 -0.0000000 -3.1415926"/>
         <geometry><mesh scale="1.0 1.0 1.0" filename="${M}/bucket_vslot_bearing_2.dae"/></geometry>
         <material name="bucket_dark"/>
       </visual>
       <visual>
-        <origin xyz="0.046739 0.175998 -0.020065" rpy="0.0000000 1.5707963 0.0000000"/>
+        <origin xyz="0.046739 0.053998 -0.020065" rpy="0.0000000 1.5707963 0.0000000"/>
         <geometry><mesh scale="1.0 1.0 1.0" filename="${M}/tilt_bearing_left_1.dae"/></geometry>
         <material name="bucket_dark"/>
       </visual>
       <visual>
-        <origin xyz="-0.003261 0.175998 -0.020065" rpy="0.0000000 1.5707963 -3.1415927"/>
+        <origin xyz="-0.003261 0.053998 -0.020065" rpy="0.0000000 1.5707963 -3.1415927"/>
         <geometry><mesh scale="1.0 1.0 1.0" filename="${M}/tilt_bearing_left_4.dae"/></geometry>
         <material name="bucket_dark"/>
       </visual>
       <visual>
-        <origin xyz="0.052739 0.175998 -0.020065" rpy="0.0000000 1.5707963 0.0000000"/>
+        <origin xyz="0.052739 0.053998 -0.020065" rpy="0.0000000 1.5707963 0.0000000"/>
         <geometry><mesh scale="1.0 1.0 1.0" filename="${M}/tilt_bearing_left_2.dae"/></geometry>
         <material name="bucket_dark"/>
       </visual>
       <visual>
-        <origin xyz="-0.009261 0.175998 -0.020065" rpy="0.0000000 1.5707963 -3.1415927"/>
+        <origin xyz="-0.009261 0.053998 -0.020065" rpy="0.0000000 1.5707963 -3.1415927"/>
         <geometry><mesh scale="1.0 1.0 1.0" filename="${M}/tilt_bearing_left_3.dae"/></geometry>
         <material name="bucket_dark"/>
@@ -492,5 +496,5 @@
            link below, because they swing with it. -->
       <collision name="${prefix}bucket_body_collision">
-        <origin xyz="0.04500 0.12200 0.03300" rpy="0 0 0"/>
+        <origin xyz="0.04500 0 0.03300" rpy="0 0 0"/>
         <geometry><box size="0.010 0.460 0.145"/></geometry>
       </collision>
@@ -501,5 +505,9 @@
       <parent link="${prefix}bucket_lift_arm"/>
       <child link="${prefix}bucket_body"/>
-      <origin xyz="${arm_length} ${bucket_pivot_y} -0.00001" rpy="0 0 0"/>
+      <!-- y is 0 so bucket_body lands on the centre line. The bucket really hangs
+           off ONE arm (Revolute_2 on Square_Tube_2), 0.102 m to the right of the arm
+           pivot midpoint; that offset is carried by bucket_body's own origins. Sliding
+           this joint along its own y axis does not move the axis line. -->
+      <origin xyz="${arm_length} ${bucket_frame_y} -0.00001" rpy="0 0 0"/>
       <axis xyz="0 -1 0"/>
       <limit lower="${tilt_lower}" upper="${tilt_upper}"
@@ -521,5 +529,5 @@
       <parent link="${prefix}bucket_body"/>
       <child link="${prefix}bucket_jaw"/>
-      <origin xyz="0.076453 0.348498 0.158935" rpy="0 0 0"/>
+      <origin xyz="0.076453 0 0.158935" rpy="0 0 0"/>
       <axis xyz="0 1 0"/>
       <limit lower="${jaw_lower}" upper="${jaw_upper}"
@@ -529,5 +537,5 @@
     <link name="${prefix}bucket_jaw">
       <inertial>
-        <origin xyz="0.021080 -0.226498 -0.132757" rpy="0 0 0"/>
+        <origin xyz="0.021080 0 -0.132757" rpy="0 0 0"/>
         <mass value="${0.6777*k}"/>
         <inertia ixx="${0.024905*k}" ixy="${0.000000*k}" ixz="${0.001904*k}"
@@ -536,5 +544,5 @@
       </inertial>
       <visual>
-        <origin xyz="0.000000 0.000000 0.000000" rpy="1.5707963 0.0000000 0.0000000"/>
+        <origin xyz="0.000000 0.226498 0.000000" rpy="1.5707963 0.0000000 0.0000000"/>
         <geometry><mesh scale="1.0 1.0 1.0" filename="${M}/bucket_jaw.dae"/></geometry>
         <material name="bucket_steel"/>
@@ -545,13 +553,13 @@
            bucket-frame values minus the hinge position. -->
       <collision name="${prefix}bucket_floor_collision">
-        <origin xyz="0.04855 -0.22650 -0.19794" rpy="0 0 0"/>
+        <origin xyz="0.04855 -0.000002 -0.19794" rpy="0 0 0"/>
         <geometry><box size="0.170 0.460 0.010"/></geometry>
       </collision>
       <collision name="${prefix}bucket_side_left_collision">
-        <origin xyz="0.04855 -0.02150 -0.12294" rpy="0 0 0"/>
+        <origin xyz="0.04855 0.204998 -0.12294" rpy="0 0 0"/>
         <geometry><box size="0.170 0.049 0.150"/></geometry>
       </collision>
       <collision name="${prefix}bucket_side_right_collision">
-        <origin xyz="0.04855 -0.44450 -0.12294" rpy="0 0 0"/>
+        <origin xyz="0.04855 -0.218002 -0.12294" rpy="0 0 0"/>
         <geometry><box size="0.170 0.023 0.150"/></geometry>
       </collision>
@@ -570,8 +578,8 @@
          over the whole workspace: rod end lands within 0.01 mm. -->
     <xacro:bucket_ram name="bucket_ram_lift_left"  parent="bucket_frame" mesh="lift_ram_left"
-                      xyz="0.00004 0.119074 -0.24001"
+                      xyz="0.00004 0.099074 -0.24001"
                       mesh_rpy="0 -1.5707963 -1.5707963" axis="1 0 0" phi="0"/>
     <xacro:bucket_ram name="bucket_ram_lift_right" parent="bucket_frame" mesh="lift_ram_right"
-                      xyz="0.00004 -0.079074 -0.24001"
+                      xyz="0.00004 -0.099074 -0.24001"
                       mesh_rpy="0 -1.5707963 1.5707963" axis="1 0 0" phi="0"/>
     <!-- The tilt ram's barrel is bolted to the plate on the ARMS (the
@@ -585,14 +593,14 @@
          rather than its origin. -->
     <xacro:bucket_ram name="bucket_ram_tilt" parent="bucket_lift_arm" mesh="tilt_ram"
-                      xyz="0.18674 0.030248 0.01399"
+                      xyz="0.18674 0.010248 0.01399"
                       mesh_xyz="0.365 -0.02025 0"
                       mesh_rpy="0 1.5707963 -1.5707963" axis="1 0 0" phi="0"/>
     <!-- The two 50 mm jaw actuators. Right side is -y (act 1), left is +y (act 2). -->
-    <xacro:bucket_jaw_ram name="bucket_ram_jaw_right" y="-0.08137"
+    <xacro:bucket_jaw_ram name="bucket_ram_jaw_right" y="-0.20337"
         base_mesh="jaw_ram_right_barrel"
         shaft_mesh="jaw_ram_right_shaft"
         barrel_xyz="0 0.02287 0" barrel_rpy="0 1.5707963 -1.5707963"
         shaft_xyz="0.20681 -0.02013 0" shaft_rpy="0 1.5707963 1.5707963"/>
-    <xacro:bucket_jaw_ram name="bucket_ram_jaw_left" y="0.32537"
+    <xacro:bucket_jaw_ram name="bucket_ram_jaw_left" y="0.20337"
         base_mesh="jaw_ram_left_barrel"
         shaft_mesh="jaw_ram_left_shaft"
@@ -606,10 +614,10 @@
          apart, measured from its mesh.
          ═══════════════════════════════════════════════════════════════════ -->
-    <xacro:bucket_encoder name="bucket_lift_encoder_left"  parent="bucket_frame" xyz="0 0.1 0"/>
-    <xacro:bucket_encoder name="bucket_lift_encoder_right" parent="bucket_frame" xyz="0 -0.1 0"/>
-    <xacro:bucket_encoder name="bucket_tilt_encoder_left"  parent="bucket_lift_arm"   xyz="${arm_length} 0.100 -0.00001"/>
-    <xacro:bucket_encoder name="bucket_tilt_encoder_right" parent="bucket_lift_arm"   xyz="${arm_length} ${bucket_pivot_y} -0.00001"/>
-    <xacro:bucket_encoder name="bucket_jaw_encoder_left"   parent="bucket_body"       xyz="0.076453 0.348498 0.158935"/>
-    <xacro:bucket_encoder name="bucket_jaw_encoder_right"  parent="bucket_body"       xyz="0.076453 -0.104502 0.158935"/>
+    <xacro:bucket_encoder name="bucket_lift_encoder_left"  parent="bucket_frame" xyz="0 0.08 0"/>
+    <xacro:bucket_encoder name="bucket_lift_encoder_right" parent="bucket_frame" xyz="0 -0.12 0"/>
+    <xacro:bucket_encoder name="bucket_tilt_encoder_left"  parent="bucket_lift_arm"   xyz="${arm_length} 0.080 -0.00001"/>
+    <xacro:bucket_encoder name="bucket_tilt_encoder_right" parent="bucket_lift_arm"   xyz="${arm_length} -0.122 -0.00001"/>
+    <xacro:bucket_encoder name="bucket_jaw_encoder_left"   parent="bucket_body"       xyz="0.076453 0.226498 0.158935"/>
+    <xacro:bucket_encoder name="bucket_jaw_encoder_right"  parent="bucket_body"       xyz="0.076453 -0.226498 0.158935"/>
   </xacro:macro>
 </robot>
