Commit message: Refactor URDF and YAML configurations: update sensor properties and remove 2D LIDAR references

File: software/ros_ws/src/description/urdf/perseus.urdf.xacro (robot description, xacro)
@@ -42,8 +42,5 @@
     <xacro:property name="bar_width" value="0.03"/>
     <xacro:property name="bar_height" value="0.03"/>
-    <!-- 2D and 3D LIDAR Properties -->
-    <xacro:property name="laser_2d_mass" value="0.1"/>
-    <xacro:property name="laser_2d_radius" value="0.04"/>
-    <xacro:property name="laser_2d_length" value="0.04"/>
+    <!-- 3D LIDAR Properties -->
     <xacro:property name="livox_mass" value="0.2"/>
     <xacro:property name="livox_radius" value="0.04"/>
@@ -59,6 +56,8 @@
     <xacro:property name="sensor_mount_y_offset" value="0.0"/>
     <xacro:property name="sensor_mount_z_offset" value="${chassis_height + 0.05}"/>
-    <!-- nose-down tilt of the Livox: positive pitch swings its +x axis towards -z -->
-    <xacro:property name="livox_pitch" value="${pi/4}"/>
+    <!-- nose-down tilt of the Livox base plate, applied at livox_base_joint in
+         sensor_mount.urdf.xacro: positive pitch swings its +x axis towards -z. The
+         sensor is fixed to the plate, so this aims the LiDAR. Zero leaves it level. -->
+    <xacro:property name="lidar_angle" value="${pi/4}"/>
     <!-- ADD COMPONENTS -->
     <xacro:include filename="$(find description)/urdf/inertia_macros.xacro"/>
@@ -95,9 +94,4 @@
     <!-- Livox and RealSense both hang off the mast: see sensor_mount.urdf.xacro -->
     <xacro:sensor_mount prefix="${prefix}"/>
-    <joint name="${prefix}laser_2d_joint" type="fixed">
-      <parent link="${prefix}chassis"/>
-      <child link="${prefix}laser_2d_frame"/>
-      <origin xyz="-0.15 0 0.25" rpy="0 0 0"/>
-    </joint>
   </xacro:macro>
 </robot>

File: software/ros_ws/src/description/urdf/sensor_mount.urdf.xacro (robot description, xacro)
@@ -7,6 +7,6 @@
     extends backwards in -x and upwards in +z from that origin. "Front of the chassis,
     a bit above" is therefore x near 0 and z a little over chassis_height.
-    Both sensors hang off sensor_mount rather than off chassis, so re-siting the mast
-    only means changing sensor_mount_*_offset.
+    Both sensors hang off sensor_mount rather than off chassis (the Livox through
+    livox_base), so re-siting the mast only means changing sensor_mount_*_offset.
   -->
   <xacro:macro name="sensor_mount" params="prefix:=^">
@@ -30,13 +30,59 @@
     </joint>
     <!--
-      Livox MID-360, on top of the mast and pitched nose-down by livox_pitch.
-      A positive pitch about +y takes the sensor +x axis towards -z, so this points the
-      LiDAR forwards and down. The IMU-LiDAR extrinsic in the fast_lio config is internal
-      to the sensor housing and is unaffected by how the housing is mounted.
+      Plate on top of the mast that the Livox bolts onto. lidar_angle is applied here, and
+      the sensor is fixed to the plate, so the two tilt together: a positive pitch about +y
+      takes the plate, and with it the sensor +x axis, towards -z, pointing the LiDAR
+      forwards and down. Re-aiming the LiDAR means changing lidar_angle and nothing else.
+    -->
+    <link name="${prefix}livox_base">
+      <!-- no mesh for the plate yet: a visual without a geometry fails to parse, so the
+           whole element stays commented out until there is one to point at.
+      <visual>
+        <origin xyz="0.0 0.0 0.0" rpy="0.0 0.0 ${pi/2}"/>
+        <geometry>
+          <mesh scale="1.0 1.0 1.0" filename="file://$(find description)/meshes/sensor_mount.dae"/>
+        </geometry>
+      </visual>
+      -->
+    </link>
+    <joint name="${prefix}livox_base_joint" type="fixed">
+      <parent link="${prefix}sensor_mount"/>
+      <child link="${prefix}livox_base"/>
+      <origin xyz="0.024 0.0 0.061" rpy="0.0 ${lidar_angle} 0.0"/>
+    </joint>
+    <!--
+      Livox MID-360 itself. The mesh and the collision cylinder are offset down by 20 mm
+      because the sensor frame sits above the housing floor; the rpy on the visual only
+      aligns the exported mesh with that frame.
+    -->
+    <link name="${prefix}livox_frame">
+      <inertial>
+        <origin xyz="0 0.0 0.0" rpy="${pi/2} 0.0 ${pi}"/>
+        <mass value="${livox_mass}"/>
+        <xacro:box_inertia m="${livox_mass}" x="${livox_length}" y="${livox_radius}" z="${livox_radius}"/>
+      </inertial>
+      <visual>
+        <origin xyz="0 0.0 -0.02" rpy="${pi/2} 0.0 ${pi}"/>
+        <geometry>
+          <mesh scale="1.0 1.0 1.0" filename="file://$(find description)/meshes/mid-360.dae"/>
+        </geometry>
+      </visual>
+      <collision>
+        <origin xyz="0 0.0 -0.02" rpy="0.0 0.0 0.0"/>
+        <geometry>
+          <cylinder radius="${livox_radius}" length="${livox_length}"/>
+        </geometry>
+      </collision>
+    </link>
+    <!--
+      Livox MID-360, seated on livox_base. The joint only offsets it across the plate and
+      adds no rotation of its own, so the sensor inherits the plate's tilt. The IMU-LiDAR
+      extrinsic in the fast_lio config is internal to the sensor housing and is unaffected
+      by how the housing is mounted.
     -->
     <joint name="${prefix}laser_joint" type="fixed">
-      <parent link="${prefix}sensor_mount"/>
+      <parent link="${prefix}livox_base"/>
       <child link="${prefix}livox_frame"/>
-      <origin xyz="0.04 0.0 0.13" rpy="${-livox_pitch} 0.0 ${0.0}"/>
+      <origin xyz="${-0.08} 0.0 0.05" rpy="${0.0} 0.0 ${0.0}"/>
     </joint>
     <!-- RealSense D455, on the front face of the mast, looking straight ahead -->

File: software/ros_ws/src/description/urdf/sensors.urdf.xacro (robot description, xacro)
@@ -1,46 +1,9 @@
 <?xml version="1.0"?>
 <robot name="lidar" xmlns:xacro="http://ros.org/wiki/xacro">
-<!-- 3D LIDAR (Existing - Livox MID-360) -->
-<link name="${prefix}livox_frame">
-    <inertial>
-        <origin xyz="0 0.0 0.0" rpy="${pi/2} 0.0 ${pi}"/>
-        <mass value="${livox_mass}"/>
-        <xacro:box_inertia m="${livox_mass}" x="${livox_length}" y="${livox_radius}" z="${livox_radius}"/>
-    </inertial>
-    <visual>
-        <origin xyz="0 0.0 -0.02" rpy="${pi/2} 0.0 ${pi}"/>
-        <geometry>
-            <mesh scale="1.0 1.0  1.0" filename="file://$(find description)/meshes/mid-360.dae"/>
-        </geometry>
-    </visual>
-    <collision>
-        <origin xyz="0 0.0 -0.02" rpy="0.0 0.0 0.0"/>
-        <geometry>
-            <cylinder radius="${livox_radius}" length="${livox_length}"/>
-        </geometry>
-    </collision>
-</link>
-<!-- 2D LIDAR -->
-<link name="${prefix}laser_2d_frame">
-    <inertial>
-        <origin xyz="0 0 0"/>
-        <mass value="${laser_2d_mass}"/>
-        <xacro:box_inertia m="${laser_2d_mass}" x="${laser_2d_length}" y="${laser_2d_radius}" z="${laser_2d_radius}"/>
-    </inertial>
-    <visual>
-        <origin xyz="0 0 0"/>
-        <geometry>
-            <cylinder radius="${laser_2d_radius}" length="${laser_2d_length}"/>
-        </geometry>
-        <material name="blue">
-            <color rgba="0.0 0.0 1.0 1.0"/>
-        </material>
-    </visual>
-    <collision>
-        <geometry>
-            <cylinder radius="0.04" length="0.04"/>
-        </geometry>
-    </collision>
-</link>
+<!--
+  Gazebo-only description of the Livox MID-360: the gpu_lidar that stands in for the
+  scanner and the IMU inside the housing. The livox_frame link they attach to is part
+  of the mast, so it lives in sensor_mount.urdf.xacro next to the joint that aims it.
+-->
 <!-- Simulating the Livox MID-360 -->
 <gazebo reference="${prefix}livox_frame">
@@ -79,40 +42,4 @@
   </sensor>
 </gazebo>
-<!-- 2D LIDAR SENSOR (Traditional 2D Laser Scanner) -->
-<gazebo reference="${prefix}laser_2d_frame">
-  <material>
-    <ambient>0.0 0.0 1.0 1</ambient>
-    <diffuse>0.0 0.0 1.0 1</diffuse>
-    <specular>0.0 0.0 1.0 1</specular>
-  </material>
-  <sensor name="${prefix}laser_2d_sensor" type="gpu_lidar">
-    <topic>scan</topic>
-    <update_rate>10</update_rate>
-    <always_on>true</always_on>
-    <visualize>false</visualize>
-    <ray>
-      <scan>
-        <horizontal>
-          <samples>720</samples>
-          <resolution>1</resolution>
-          <min_angle>-3.14159</min_angle>
-          <max_angle>3.14159</max_angle>
-        </horizontal>
-        <!-- Single horizontal plane for 2D scanning -->
-        <vertical>
-          <samples>1</samples>
-          <min_angle>0.0</min_angle>
-          <max_angle>0.0</max_angle>
-        </vertical>
-      </scan>
-      <range>
-        <min>0.05</min>
-        <max>200.0</max>
-        <resolution>0.01</resolution>
-      </range>
-    </ray>
-    <gz_frame_id>${prefix}laser_2d_frame</gz_frame_id>
-  </sensor>
-</gazebo>
 <gazebo reference="${prefix}livox_frame">
     <material>Gazebo/Grey</material>

Commit message: fix: Correct chassis joint origin position in perseus.urdf.xacro

File: software/ros_ws/src/description/urdf/perseus.urdf.xacro (robot description, xacro)
@@ -75,5 +75,5 @@
     <link name="${prefix}base_link"/>
     <joint name="${prefix}chassis_joint" type="fixed"> <!-- Joint Connect base_link and chassis -->
-      <origin xyz="${0.2} 0.0 ${chassis_z_offset}" rpy="0.0 0.0 0.0"/>
+      <origin xyz="${0.0} 0.0 ${chassis_z_offset}" rpy="0.0 0.0 0.0"/>
       <parent link="${prefix}base_link"/>
       <child link="${prefix}chassis"/>

Commit message: fix: Adjust sensor mount y offset and update lidar angle for improved sensor alignment

File: software/ros_ws/src/description/urdf/perseus.urdf.xacro (robot description, xacro)
@@ -54,10 +54,10 @@
          front and z above chassis_height clears the deck -->
     <xacro:property name="sensor_mount_x_offset" value="0.0"/>
-    <xacro:property name="sensor_mount_y_offset" value="0.0"/>
+    <xacro:property name="sensor_mount_y_offset" value="0.015"/>
     <xacro:property name="sensor_mount_z_offset" value="${chassis_height + 0.05}"/>
     <!-- nose-down tilt of the Livox base plate, applied at livox_base_joint in
          sensor_mount.urdf.xacro: positive pitch swings its +x axis towards -z. The
          sensor is fixed to the plate, so this aims the LiDAR. Zero leaves it level. -->
-    <xacro:property name="lidar_angle" value="${pi/4}"/>
+    <xacro:property name="lidar_angle" value="${7*pi/36}"/>
     <!-- ADD COMPONENTS -->
     <xacro:include filename="$(find description)/urdf/inertia_macros.xacro"/>
