Commit message: Implement low-speed stall mitigation with PID controller and configuration updates

File: software/ros_ws/src/description/ros2_control/perseus.ros2_control.xacro (robot description, xacro)
@@ -1,5 +1,5 @@
 <?xml version="1.0"?>
 <robot xmlns:xacro="http://www.ros.org/wiki/xacro">
-  <xacro:macro name="perseus_ros2_control" params="namespace:='' name prefix can_bus:='can0' hardware_plugin">
+  <xacro:macro name="perseus_ros2_control" params="namespace:='' name prefix can_bus:='can0' hardware_plugin min_command_erpm:='0'">
     <ros2_control name="${name}" type="system">
       <hardware>
@@ -8,4 +8,7 @@
         <!-- Enable velocity -> position integration over time for mock hardware -->
         <param name="calculate_dynamics">true</param>
+        <!-- Speed floor for the ESCs, in ERPM; 0 leaves commands untouched.
+             See VescSystemHardware::_min_command_erpm. -->
+        <param name="min_command_erpm">${min_command_erpm}</param>
       </hardware>
       <xacro:macro name="ros2_control_joint" params="name id">

File: software/ros_ws/src/perseus/urdf/perseus.urdf.xacro (robot description, xacro)
@@ -4,4 +4,5 @@
   <xacro:arg name="can_bus" default="can0" />
   <xacro:arg name="hardware_plugin" default="hardware/VescSystemHardware" />
+  <xacro:arg name="min_command_erpm" default="0" />
   <!-- Import URDF description -->
   <xacro:include filename="$(find description)/urdf/perseus.urdf.xacro" />
@@ -12,4 +13,4 @@
   <!-- Instantiate the description and the ROS2 control information -->
   <xacro:perseus prefix="$(arg prefix)" />
-  <xacro:perseus_ros2_control name="Perseus" prefix="$(arg prefix)" can_bus="$(arg can_bus)" hardware_plugin="$(arg hardware_plugin)"/>
+  <xacro:perseus_ros2_control name="Perseus" prefix="$(arg prefix)" can_bus="$(arg can_bus)" hardware_plugin="$(arg hardware_plugin)" min_command_erpm="$(arg min_command_erpm)"/>
 </robot>
