Commit message: feat: ros2_control with urdf

File: software/ros_ws/src/description/ros2_control/bucket.ros2_control.xacro (robot description, xacro)
@@ -2,32 +2,25 @@
 <robot xmlns:xacro="http://www.ros.org/wiki/xacro">
   <!--
-    Include this file from the main URDF/xacro with:
-      <xacro:include filename="$(find description)/ros2_control/bucket.ros2_control.xacro"/>
-      <xacro:bucket_ros2_control can_interface="can0"/>
-    Each joint below is tagged with "axis" and "side" - these are read by
-    BucketHardware::on_init() to decide which CAN actuator it maps to.
-    Commands are bank-level, not per-side: the CAN board deliberately only
-    accepts one setpoint per axis (independent left/right control is
-    possible in hardware but is disallowed over CAN to prevent torsion in
-    the bucket). So exactly ONE joint per axis (arbitrarily "_left" here)
-    declares a command_interface; its pair declares state_interfaces only.
-    Position is the only command interface. Speed control is the separate,
-    non-ros2_control teleop driver's job (payloads/bucket_driver) - the two
-    must never run at once, since the firmware takes its control mode from
-    whichever command arrived last.
-    BucketHardware::on_init() enforces this 1-commandable-joint-per-axis
-    invariant and will refuse to configure otherwise.
+    ros2_control block for the bucket's three driven joints (see bucket.urdf.xacro).
+    Commands are bank-level: the CAN board takes one position setpoint per axis and
+    drives both sides of that axis from it, so each axis is one joint here. The
+    "axis" and "side" params tell BucketHardware which CAN actuator a joint maps to;
+    only the left encoder of each axis is exposed for now.
+    Never run this alongside the bucket_driver teleop node. The firmware takes its
+    control mode (speed or position) from whichever command arrived last.
+    hardware_plugin can be set to mock_components/GenericSystem to exercise
+    controllers without the bucket fitted.
   -->
-  <xacro:macro name="bucket_ros2_control" params="can_interface:='can0'">
+  <xacro:macro name="bucket_ros2_control"
+      params="prefix:='' can_interface:='can0' hardware_plugin:='payloads/BucketHardware'">
     <ros2_control name="BucketSystem" type="system">
       <hardware>
-        <plugin>payloads/BucketHardware</plugin>
+        <plugin>${hardware_plugin}</plugin>
         <param name="can_interface">${can_interface}</param>
       </hardware>
-      <!-- The one joint per axis that actually receives commands. -->
-      <xacro:macro name="bucket_command_joint" params="joint_name axis side">
-        <joint name="${joint_name}">
+      <xacro:macro name="bucket_ros2_control_joint" params="joint axis">
+        <joint name="${prefix}${joint}">
           <param name="axis">${axis}</param>
-          <param name="side">${side}</param>
+          <param name="side">left</param>
           <command_interface name="position"/>
           <state_interface name="position"/>
@@ -36,24 +29,7 @@
         </joint>
       </xacro:macro>
-      <!--
-        Its pair: a real, independently-encoded joint (needed for
-        state/skew feedback and TF), but not independently commandable, so
-        no command_interfaces here.
-      -->
-      <xacro:macro name="bucket_state_only_joint" params="joint_name axis side">
-        <joint name="${joint_name}">
-          <param name="axis">${axis}</param>
-          <param name="side">${side}</param>
-          <state_interface name="position"/>
-          <state_interface name="velocity"/>
-          <state_interface name="effort"/>
-        </joint>
-      </xacro:macro>
-      <xacro:bucket_command_joint    joint_name="lift_left"   axis="lift" side="left"/>
-      <xacro:bucket_state_only_joint joint_name="lift_right"  axis="lift" side="right"/>
-      <xacro:bucket_command_joint    joint_name="tilt_left"   axis="tilt" side="left"/>
-      <xacro:bucket_state_only_joint joint_name="tilt_right"  axis="tilt" side="right"/>
-      <xacro:bucket_command_joint    joint_name="jaws_left"   axis="jaws" side="left"/>
-      <xacro:bucket_state_only_joint joint_name="jaws_right"  axis="jaws" side="right"/>
+      <xacro:bucket_ros2_control_joint joint="bucket_lift_joint" axis="lift"/>
+      <xacro:bucket_ros2_control_joint joint="bucket_tilt_joint" axis="tilt"/>
+      <xacro:bucket_ros2_control_joint joint="bucket_jaw_joint" axis="jaws"/>
     </ros2_control>
   </xacro:macro>

File: software/ros_ws/src/payloads/urdf/bucket_standalone.urdf.xacro (robot description, xacro)
@@ -1,29 +1,20 @@
 <?xml version="1.0"?>
 <!--
-  Minimal robot description for running the bucket's own controller_manager.
-  The payload gets its own controller_manager in the `payloads` namespace
-  rather than joining the drive base's, because a payload is optional and
-  hot-swappable and the base must not fail to start when no bucket is fitted.
-  That manager still needs a robot_description containing the bucket's
-  <ros2_control> block, which is what this wrapper provides.
-  bucket.ros2_control.xacro only *defines* the macro, so it has to be
-  instantiated here - running xacro on it directly yields an empty <robot/>.
-  Note this describes no links or joints, only the ros2_control block. TF for
-  the bucket comes from the full robot URDF in the `description` package, which
-  should include the same fragment. Keeping one copy of the fragment in
-  `description` is what stops the two drifting apart.
+  Robot description for the bucket's own controller_manager in the `payloads`
+  namespace. The payload is optional and hot-swappable, so it does not join the
+  drive base's controller_manager.
+  Jazzy's controller_manager reads robot_description from a topic published by
+  robot_state_publisher, which rejects a URDF with no links, so the real bucket
+  geometry is included here. The bucket macro parents bucket_mount to `chassis`,
+  so a bare `chassis` link is the root.
 -->
 <robot xmlns:xacro="http://www.ros.org/wiki/xacro" name="bucket">
   <xacro:arg name="can_interface" default="can0"/>
-  <!--
-    robot_state_publisher rejects a URDF with no links, and Jazzy's
-    controller_manager needs it to publish the robot_description topic - so a
-    kinematic model is mandatory even for a headless control stack. The one
-    included here is PLACEHOLDER geometry; see the warning in bucket.urdf.xacro.
-  -->
-  <link name="bucket_base"/>
+  <xacro:arg name="hardware_plugin" default="payloads/BucketHardware"/>
+  <link name="chassis"/>
+  <xacro:include filename="$(find description)/urdf/inertia_macros.xacro"/>
   <xacro:include filename="$(find description)/urdf/bucket.urdf.xacro"/>
-  <xacro:bucket_description parent="bucket_base"/>
+  <xacro:bucket prefix=""/>
   <xacro:include filename="$(find description)/ros2_control/bucket.ros2_control.xacro"/>
-  <xacro:bucket_ros2_control can_interface="$(arg can_interface)"/>
+  <xacro:bucket_ros2_control can_interface="$(arg can_interface)" hardware_plugin="$(arg hardware_plugin)"/>
 </robot>

Commit message: feat: Code ready for testin

File: software/ros_ws/src/description/ros2_control/bucket.ros2_control.xacro (robot description, xacro)
@@ -11,4 +11,9 @@
     hardware_plugin can be set to mock_components/GenericSystem to exercise
     controllers without the bucket fitted.
+    offset_deg and direction map the firmware's angle onto the URDF joint:
+      joint_deg = direction * (firmware_deg - offset_deg)
+    Joint conventions (bucket.urdf.xacro): lift 0 at highest, positive down; tilt
+    0 level, positive dumping; jaw 0 closed, positive opening. Leave the defaults
+    when the firmware calibration already matches them.
   -->
   <xacro:macro name="bucket_ros2_control"
@@ -19,8 +24,10 @@
         <param name="can_interface">${can_interface}</param>
       </hardware>
-      <xacro:macro name="bucket_ros2_control_joint" params="joint axis">
+      <xacro:macro name="bucket_ros2_control_joint" params="joint axis offset_deg:=0.0 direction:=1">
         <joint name="${prefix}${joint}">
           <param name="axis">${axis}</param>
           <param name="side">left</param>
+          <param name="offset_deg">${offset_deg}</param>
+          <param name="direction">${direction}</param>
           <command_interface name="position"/>
           <state_interface name="position"/>

File: software/ros_ws/src/description/urdf/bucket.urdf.xacro (robot description, xacro)
@@ -54,5 +54,6 @@
        sit 6.24 deg below the frame's own x axis - they never quite reach
        horizontal. Joint zero is placed at full extension (top of travel,
-       transport pose) by baking that 6.24 deg into the joint origin.
+       transport pose) by baking that 6.24 deg into the joint origin, and the
+       joint counts positive DOWN from there: 0 .. 71.36 deg.
        Worth knowing: the CAD's *exported* pose needs L = 0.640, which is 25 mm
        beyond full extension. That is not an error in the CAD - the toolkit
@@ -73,6 +74,7 @@
   <!-- nose-down pitch of the arm at joint zero, relative to the frame -->
   <xacro:property name="lift_zero_pitch" value="${-(asin(lift_sin_ext) - lift_phase)}"/>
-  <xacro:property name="lift_lower" value="${asin(lift_sin_ret) - asin(lift_sin_ext)}"/>
-  <xacro:property name="lift_upper" value="0.0"/>
+  <xacro:property name="lift_lower" value="0.0"/>
+  <!-- 71.36 deg -->
+  <xacro:property name="lift_upper" value="${asin(lift_sin_ext) - asin(lift_sin_ret)}"/>
   <!-- ══ Tilt travel ═════════════════════════════════════════════════════
        Same treatment. The tilt actuator works between a pin on the bucket
@@ -85,7 +87,9 @@
        Curl is capped short of that fold: past about 1.6 rad the bucket is
        folded back over the arms, which the real structure will not allow.
-       Dump is the true actuator limit. -->
-  <xacro:property name="tilt_lower" value="-0.490398"/>
-  <xacro:property name="tilt_upper" value="1.600000"/>
+       Dump is the true actuator limit.
+       The joint counts positive toward DUMP (tipping down) from the CAD pose,
+       so curl is negative: -91.673 (curl) .. +28.098 (dump) deg. -->
+  <xacro:property name="tilt_lower" value="${radians(-91.673)}"/>
+  <xacro:property name="tilt_upper" value="${radians(28.098)}"/>
   <!-- geometric, for reference -->
   <xacro:property name="tilt_fold_limit" value="1.889229"/>
@@ -119,7 +123,9 @@
            extended end (CAD pose) : theta =  0.0000
            retracted end           : theta = -0.8376   (L falls by 50 mm)
-       (The other reading would give 0 .. +1.0540; it does not apply.) -->
-  <xacro:property name="jaw_lower" value="-0.8376"/>
-  <xacro:property name="jaw_upper" value="0.0"/>
+       (The other reading would give 0 .. +1.0540; it does not apply.)
+       The joint is -theta, so it counts positive OPENING from closed:
+       0 .. 47.991 deg. -->
+  <xacro:property name="jaw_lower" value="0.0"/>
+  <xacro:property name="jaw_upper" value="${radians(47.991)}"/>
   <xacro:property name="jaw_moment_arm" value="0.0615"/>
   <xacro:property name="jaw_effort" value="${actuator_force*jaw_moment_arm}"/>
@@ -395,5 +401,5 @@
       </collision>
     </link>
-    <!-- Positive raises. Zero is the top of travel, with the arms 6.24 deg
+    <!-- Positive lowers. Zero is the top of travel, with the arms 6.24 deg
          below the frame axis because that is as far as the actuators reach. -->
     <joint name="${prefix}bucket_lift_joint" type="revolute">
@@ -401,5 +407,5 @@
       <child link="${prefix}bucket_lift_arm"/>
       <origin xyz="0 0 0" rpy="0 ${lift_zero_pitch} 0"/>
-      <axis xyz="0 -1 0"/>
+      <axis xyz="0 1 0"/>
       <limit lower="${lift_lower}" upper="${lift_upper}"
              effort="${lift_effort}" velocity="${lift_velocity}"/>
@@ -505,6 +511,6 @@
       </collision>
     </link>
-    <!-- Positive curls the scoop back to retain a load; negative dumps.
-         Zero is the CAD pose. -->
+    <!-- Positive dumps (tips down); negative curls the scoop back to retain a
+         load. Zero is the CAD pose, taken as level. -->
     <joint name="${prefix}bucket_tilt_joint" type="revolute">
       <parent link="${prefix}bucket_lift_arm"/>
@@ -515,5 +521,5 @@
            this joint along its own y axis does not move the axis line. -->
       <origin xyz="${arm_length} ${bucket_frame_y} -0.00001" rpy="0 0 0"/>
-      <axis xyz="0 -1 0"/>
+      <axis xyz="0 1 0"/>
       <limit lower="${tilt_lower}" upper="${tilt_upper}"
              effort="${tilt_effort}" velocity="${tilt_velocity}"/>
@@ -526,6 +532,7 @@
          is the hinge, frame-aligned, so the joint origin is simply the hinge
          position measured from the tilt pivot.
-         Positive closes (the tray swings back toward the REAR half), negative
-         opens; zero is the CAD pose. The axis is the CAD mate's own axis.
+         Positive opens, negative closes (the tray swings back toward the REAR
+         half); zero is the CAD pose, fully closed. The axis is the CAD mate's
+         axis, reversed so opening counts positive.
          The rod ends of the two 50 mm actuators pin to this half; the rods
          themselves are the animated "Jaw rams" links, not part of this one.
@@ -535,5 +542,5 @@
       <child link="${prefix}bucket_jaw"/>
       <origin xyz="0.076453 0 0.158935" rpy="0 0 0"/>
-      <axis xyz="0 1 0"/>
+      <axis xyz="0 -1 0"/>
       <limit lower="${jaw_lower}" upper="${jaw_upper}"
              effort="${jaw_effort}" velocity="${jaw_velocity}"/>

Commit message: feat: Osciallation fix

File: software/ros_ws/src/description/ros2_control/bucket.ros2_control.xacro (robot description, xacro)
@@ -22,4 +22,11 @@
     0 level, positive dumping; jaw 0 closed, positive opening. Leave the defaults
     when the firmware calibration already matches them.
+    hold_deg and resume_deg are a hold deadband, in joint degrees; 0 leaves it off.
+    Within hold_deg of a setpoint that has stopped moving, BucketHardware stops the
+    bank and sends nothing until the setpoint changes or the joint drifts past
+    resume_deg. The firmware's own full-duty position loop otherwise hunts around
+    the setpoint when the joint coasts past its 2-3 deg window. Keep the
+    controller's goal tolerance (bucket_controller.yaml) at least hold_deg, or a
+    goal can stop short of it and never succeed.
   -->
   <xacro:macro name="bucket_ros2_control"
@@ -30,9 +37,11 @@
         <param name="can_interface">${can_interface}</param>
       </hardware>
-      <xacro:macro name="bucket_ros2_control_joint" params="joint axis offset_deg:=0.0 direction:=1">
+      <xacro:macro name="bucket_ros2_control_joint" params="joint axis offset_deg:=0.0 direction:=1 hold_deg:=0.0 resume_deg:=0.0">
         <joint name="${prefix}${joint}">
           <param name="axis">${axis}</param>
           <param name="offset_deg">${offset_deg}</param>
           <param name="direction">${direction}</param>
+          <param name="hold_deg">${hold_deg}</param>
+          <param name="resume_deg">${resume_deg}</param>
           <command_interface name="position"/>
           <state_interface name="position"/>
@@ -43,5 +52,6 @@
       <xacro:bucket_ros2_control_joint joint="bucket_lift_joint" axis="lift"/>
       <xacro:bucket_ros2_control_joint joint="bucket_tilt_joint" axis="tilt"/>
-      <xacro:bucket_ros2_control_joint joint="bucket_jaw_joint" axis="jaws"/>
+      <xacro:bucket_ros2_control_joint joint="bucket_jaw_joint" axis="jaws"
+          hold_deg="2.5" resume_deg="6.0"/>
     </ros2_control>
   </xacro:macro>
