Commit message: fix(arm_model): change shoulder_pan joint type to revolute and update limits

File: software/ros_ws/src/payloads/config/arm_model.urdf (robot description, URDF)
Before this commit: robot arm, 11 links, 10 joints
Joints:
- joint shoulder_pan: limit effort=10.0 velocity=2.0 -> lower=-31.4159 upper=31.4159 effort=10.0 velocity=3.0; type continuous -> revolute
