Commit message: Integrate 3-DOF arm teleoperation simulation

File: software/ros_ws/src/payloads/config/arm.ros2_control.xacro (robot description, xacro)
@@ -1,14 +1,24 @@
 <?xml version="1.0"?>
 <robot xmlns:xacro="http://www.ros.org/wiki/xacro">
-    <xacro:macro name="arm_ros2_control" params="name initial_positions_file">
+    <xacro:macro name="arm_ros2_control" params="name initial_positions_file use_mock_hardware:=false hardware_plugin:=mock_components/GenericSystem port:=/dev/ttyUSB0 baud_rate:=1000000">
         <xacro:property name="initial_positions" value="${xacro.load_yaml(initial_positions_file)['initial_positions']}"/>
         <ros2_control name="${name}" type="system">
             <hardware>
-                <!-- Step 2 intentionally supports mock hardware only. -->
-                <plugin>mock_components/GenericSystem</plugin>
+                <!--
+                     use_mock_hardware:=true for simulation, or point the
+                     hardware_plugin at your own servo hardware_interface plugin.
+                     use_mock_hardware:=false  -->
+                <xacro:if value="${use_mock_hardware}">
+                  <plugin>mock_components/GenericSystem</plugin>
+                </xacro:if>
+                <xacro:unless value="${use_mock_hardware}">
+                  <plugin>${hardware_plugin}</plugin>
+                  <param name="port">${port}</param>
+                  <param name="baud_rate">${baud_rate}</param>
+                </xacro:unless>
             </hardware>
             <joint name="shoulder_tilt">
+                <param name="id">2</param>
                 <command_interface name="position"/>
-                <command_interface name="velocity"/>
                 <state_interface name="position">
                   <param name="initial_value">${initial_positions['shoulder_tilt']}</param>
@@ -17,6 +27,6 @@
             </joint>
             <joint name="shoulder_pan">
+                <param name="id">1</param>
                 <command_interface name="position"/>
-                <command_interface name="velocity"/>
                 <state_interface name="position">
                   <param name="initial_value">${initial_positions['shoulder_pan']}</param>
@@ -25,6 +35,6 @@
             </joint>
             <joint name="elbow">
+                <param name="id">3</param>
                 <command_interface name="position"/>
-                <command_interface name="velocity"/>
                 <state_interface name="position">
                   <param name="initial_value">${initial_positions['elbow']}</param>
@@ -33,6 +43,6 @@
             </joint>
             <joint name="wrist_pitch">
+                <param name="id">4</param>
                 <command_interface name="position"/>
-                <command_interface name="velocity"/>
                 <state_interface name="position">
                   <param name="initial_value">${initial_positions['wrist_pitch']}</param>
@@ -41,6 +51,6 @@
             </joint>
             <joint name="wrist_roll">
+                <param name="id">5</param>
                 <command_interface name="position"/>
-                <command_interface name="velocity"/>
                 <state_interface name="position">
                   <param name="initial_value">${initial_positions['wrist_roll']}</param>
@@ -48,12 +58,60 @@
                 <state_interface name="velocity"/>
             </joint>
-            <joint name="fake_dof">
+            <!-- right_finger_joint is a URDF mimic; ros2_control mirrors it. -->
+            <joint name="left_finger_joint">
+                <param name="id">6</param>
                 <command_interface name="position"/>
-                <command_interface name="velocity"/>
                 <state_interface name="position">
-                  <param name="initial_value">${initial_positions['fake_dof']}</param>
+                  <param name="initial_value">${initial_positions['left_finger_joint']}</param>
                 </state_interface>
                 <state_interface name="velocity"/>
             </joint>
+            <transmission name="shoulder_pan_drive">
+                <plugin>transmission_interface/SimpleTransmission</plugin>
+                <joint name="shoulder_pan" role="joint1">
+                    <mechanical_reduction>1.0</mechanical_reduction>
+                    <offset>0.0</offset>
+                </joint>
+                <actuator name="shoulder_pan_servo" role="actuator1">
+                    <mechanical_reduction>1.0</mechanical_reduction>
+                </actuator>
+            </transmission>
+            <transmission name="shoulder_tilt_drive">
+                <plugin>transmission_interface/SimpleTransmission</plugin>
+                <joint name="shoulder_tilt" role="joint1">
+                    <mechanical_reduction>1.0</mechanical_reduction>
+                    <offset>0.0</offset>
+                </joint>
+                <actuator name="shoulder_tilt_servo" role="actuator1">
+                    <mechanical_reduction>1.0</mechanical_reduction>
+                </actuator>
+            </transmission>
+            <transmission name="elbow_drive">
+                <plugin>transmission_interface/SimpleTransmission</plugin>
+                <joint name="elbow" role="joint1">
+                    <mechanical_reduction>1.0</mechanical_reduction>
+                    <offset>0.0</offset>
+                </joint>
+                <actuator name="elbow_servo" role="actuator1">
+                    <mechanical_reduction>1.0</mechanical_reduction>
+                </actuator>
+            </transmission>
+            <transmission name="wrist_differential">
+                <plugin>transmission_interface/DifferentialTransmission</plugin>
+                <joint name="wrist_pitch" role="joint1">
+                    <mechanical_reduction>1.0</mechanical_reduction>
+                    <offset>0.0</offset>
+                </joint>
+                <joint name="wrist_roll" role="joint2">
+                    <mechanical_reduction>1.0</mechanical_reduction>
+                    <offset>0.0</offset>
+                </joint>
+                <actuator name="wrist_servo_a" role="actuator1">
+                    <mechanical_reduction>1.0</mechanical_reduction>
+                </actuator>
+                <actuator name="wrist_servo_b" role="actuator2">
+                    <mechanical_reduction>1.0</mechanical_reduction>
+                </actuator>
+            </transmission>
         </ros2_control>
     </xacro:macro>

File: software/ros_ws/src/payloads/config/arm.urdf.xacro (robot description, xacro)
@@ -2,8 +2,12 @@
 <robot xmlns:xacro="http://www.ros.org/wiki/xacro" name="arm">
     <xacro:arg name="initial_positions_file" default="initial_positions.yaml" />
+    <xacro:arg name="use_mock_hardware" default="true" />
+    <xacro:arg name="hardware_plugin" default="mock_components/GenericSystem" />
+    <xacro:arg name="port" default="/dev/ttyUSB0" />
+    <xacro:arg name="baud_rate" default="1000000" />
     <!-- Import arm urdf file -->
     <xacro:include filename="$(find payloads)/config/arm_model.urdf" />
     <!-- Import control_xacro -->
     <xacro:include filename="arm.ros2_control.xacro" />
-    <xacro:arm_ros2_control name="ArmMockSystem" initial_positions_file="$(arg initial_positions_file)"/>
+    <xacro:arm_ros2_control name="DynamixelServos" initial_positions_file="$(arg initial_positions_file)" use_mock_hardware="$(arg use_mock_hardware)" hardware_plugin="$(arg hardware_plugin)" port="$(arg port)" baud_rate="$(arg baud_rate)"/>
 </robot>

File: software/ros_ws/src/payloads/config/arm_model.urdf (robot description, URDF)
Before this commit: robot arm, 9 links, 8 joints
Links:
- removed link end_effector
- removed link fake_dof_link
- added link grasp_link
- added link gripper_base, mass 0.05; collision box size=0.035 0.035 0.022; visual box size=0.035 0.035 0.022
- added link left_finger, mass 0.012; collision box size=0.01 0.008 0.04; visual box size=0.01 0.008 0.04
- added link right_finger, mass 0.012; collision box size=0.01 0.008 0.04; visual box size=0.01 0.008 0.04
- link forearm_tip: geometry visual sphere radius=0.01
- link wrist_pitch_link: geometry collision box size=0.04 0.05 0.028; visual box size=0.04 0.05 0.028
- link wrist_roll_link: mass 0.15 -> 0.05; geometry collision box size=0.035 0.035 0.006; visual box size=0.035 0.035 0.006
Joints:
- removed joint end_effector_mount
- removed joint fake_dof
- added joint grasp_frame: type fixed, parent gripper_base, child grasp_link, origin xyz=0 0 0.045 rpy=0 0 0
- added joint gripper_mount: type fixed, parent wrist_roll_link, child gripper_base, origin xyz=0 0 0.006 rpy=0 0 0
- added joint left_finger_joint: type prismatic, parent gripper_base, child left_finger, origin xyz=0 0.004 0.022 rpy=0 0 0, axis 0 1 0, limit lower=0.0 upper=0.015 effort=20.0 velocity=0.1
- added joint right_finger_joint: type prismatic, parent gripper_base, child right_finger, origin xyz=0 -0.004 0.022 rpy=0 0 0, axis 0 -1 0, limit lower=0.0 upper=0.015 effort=20.0 velocity=0.1, mimic joint=left_finger_joint multiplier=1.0 offset=0.0
- joint wrist_roll: limit lower=-3.14159 upper=3.14159 effort=10.0 velocity=2.0 -> lower=-6.28318 upper=6.28318 effort=10.0 velocity=2.0; origin xyz=0 0 0.04 rpy=0 0 0 -> xyz=0 0 0.028 rpy=0 0 0

Commit message: Add Dynamixel controller and URDF to OpenRAVE conversion scripts
- Implemented `urdf_to_openrave.py` to convert URDF files to OpenRAVE XML format for the base to end-effector chain.
- Created `dynamixel_controller.cpp` and `dynamixel_controller.hpp` to manage communication with Dynamixel servos, including torque control and position management.
- Developed `dynamixel_servos.cpp` to integrate the Dynamixel controller with the ROS hardware interface, handling joint transformations and actuator commands.
- Added support for mocking servo IDs for testing purposes without physical hardware.

File: software/ros_ws/src/payloads/config/arm.ros2_control.xacro (robot description, xacro)
@@ -1,12 +1,8 @@
 <?xml version="1.0"?>
 <robot xmlns:xacro="http://www.ros.org/wiki/xacro">
-    <xacro:macro name="arm_ros2_control" params="name initial_positions_file use_mock_hardware:=false hardware_plugin:=mock_components/GenericSystem port:=/dev/ttyUSB0 baud_rate:=1000000">
+    <xacro:macro name="arm_ros2_control" params="name initial_positions_file use_mock_hardware:=false hardware_plugin:=payloads/DynamixelServos device:=/dev/ttyUSB0 mock_servo_ids:=''">
         <xacro:property name="initial_positions" value="${xacro.load_yaml(initial_positions_file)['initial_positions']}"/>
         <ros2_control name="${name}" type="system">
             <hardware>
-                <!--
-                     use_mock_hardware:=true for simulation, or point the
-                     hardware_plugin at your own servo hardware_interface plugin.
-                     use_mock_hardware:=false  -->
                 <xacro:if value="${use_mock_hardware}">
                   <plugin>mock_components/GenericSystem</plugin>
@@ -14,10 +10,15 @@
                 <xacro:unless value="${use_mock_hardware}">
                   <plugin>${hardware_plugin}</plugin>
-                  <param name="port">${port}</param>
-                  <param name="baud_rate">${baud_rate}</param>
+                  <param name="device">${device}</param>
+                  <!-- A 6-servo read plus write at 57600 does not fit the 100 Hz
+                       controller_manager budget; at 1 Mbaud it does. -->
+                  <param name="baud_rate">1000000</param>
+                  <!-- Servo IDs simulated in software rather than addressed on
+                       the bus. Comma-separated, no spaces. -->
+                  <param name="mock_servo_ids">${mock_servo_ids}</param>
                 </xacro:unless>
             </hardware>
             <joint name="shoulder_tilt">
-                <param name="id">2</param>
+                <param name="servo_id">2</param>
                 <command_interface name="position"/>
                 <state_interface name="position">
@@ -27,5 +28,5 @@
             </joint>
             <joint name="shoulder_pan">
-                <param name="id">1</param>
+                <param name="servo_id">1</param>
                 <command_interface name="position"/>
                 <state_interface name="position">
@@ -35,5 +36,5 @@
             </joint>
             <joint name="elbow">
-                <param name="id">3</param>
+                <param name="servo_id">3</param>
                 <command_interface name="position"/>
                 <state_interface name="position">
@@ -43,5 +44,5 @@
             </joint>
             <joint name="wrist_pitch">
-                <param name="id">4</param>
+                <param name="servo_id">4</param>
                 <command_interface name="position"/>
                 <state_interface name="position">
@@ -51,5 +52,5 @@
             </joint>
             <joint name="wrist_roll">
-                <param name="id">5</param>
+                <param name="servo_id">5</param>
                 <command_interface name="position"/>
                 <state_interface name="position">
@@ -60,5 +61,9 @@
             <!-- right_finger_joint is a URDF mimic; ros2_control mirrors it. -->
             <joint name="left_finger_joint">
-                <param name="id">6</param>
+                <param name="servo_id">6</param>
+                <!-- Metres of finger travel per radian of servo 6. Placeholder:
+                     15 mm over a quarter turn. Measure with the offset in
+                     left_finger_drive before un-mocking servo 6. -->
+                <param name="prismatic_scale">0.00955</param>
                 <command_interface name="position"/>
                 <state_interface name="position">
@@ -67,4 +72,5 @@
                 <state_interface name="velocity"/>
             </joint>
+            <!-- Gearbox reductions. The hardware plugin must apply these; ros2_control only parses them. -->
             <transmission name="shoulder_pan_drive">
                 <plugin>transmission_interface/SimpleTransmission</plugin>
@@ -97,4 +103,16 @@
                 </actuator>
             </transmission>
+            <!-- offset is the servo angle (rad) at which the fingers are closed. -->
+            <transmission name="left_finger_drive">
+                <plugin>transmission_interface/SimpleTransmission</plugin>
+                <joint name="left_finger_joint" role="joint1">
+                    <mechanical_reduction>1.0</mechanical_reduction>
+                    <offset>0.0</offset>
+                </joint>
+                <actuator name="gripper_servo" role="actuator1">
+                    <mechanical_reduction>1.0</mechanical_reduction>
+                </actuator>
+            </transmission>
+            <!-- Servos 4 and 5 jointly drive pitch and roll. -->
             <transmission name="wrist_differential">
                 <plugin>transmission_interface/DifferentialTransmission</plugin>

File: software/ros_ws/src/payloads/config/arm.urdf.xacro (robot description, xacro)
@@ -3,11 +3,11 @@
     <xacro:arg name="initial_positions_file" default="initial_positions.yaml" />
     <xacro:arg name="use_mock_hardware" default="true" />
-    <xacro:arg name="hardware_plugin" default="mock_components/GenericSystem" />
-    <xacro:arg name="port" default="/dev/ttyUSB0" />
-    <xacro:arg name="baud_rate" default="1000000" />
+    <xacro:arg name="hardware_plugin" default="payloads/DynamixelServos" />
+    <xacro:arg name="device" default="/dev/ttyUSB0" />
+    <xacro:arg name="mock_servo_ids" default="" />
     <!-- Import arm urdf file -->
     <xacro:include filename="$(find payloads)/config/arm_model.urdf" />
     <!-- Import control_xacro -->
     <xacro:include filename="arm.ros2_control.xacro" />
-    <xacro:arm_ros2_control name="DynamixelServos" initial_positions_file="$(arg initial_positions_file)" use_mock_hardware="$(arg use_mock_hardware)" hardware_plugin="$(arg hardware_plugin)" port="$(arg port)" baud_rate="$(arg baud_rate)"/>
+    <xacro:arm_ros2_control name="DynamixelServos" initial_positions_file="$(arg initial_positions_file)" use_mock_hardware="$(arg use_mock_hardware)" hardware_plugin="$(arg hardware_plugin)" device="$(arg device)" mock_servo_ids="$(arg mock_servo_ids)"/>
 </robot>

Commit message: refactor: relocate dynamixel header, configure default RMW environment variables, and update arm limits and QoS

File: software/ros_ws/src/payloads/config/arm.ros2_control.xacro (robot description, xacro)
@@ -76,5 +76,5 @@
                 <plugin>hector_transmission_interface/AdjustableOffsetTransmission</plugin>
                 <joint name="shoulder_pan" role="joint1">
-                    <mechanical_reduction>3.0</mechanical_reduction>
+                    <mechanical_reduction>1.0</mechanical_reduction>
                     <offset>0.0</offset>
                 </joint>
@@ -86,5 +86,5 @@
                 <plugin>hector_transmission_interface/AdjustableOffsetTransmission</plugin>
                 <joint name="shoulder_tilt" role="joint1">
-                    <mechanical_reduction>2.5</mechanical_reduction>
+                    <mechanical_reduction>1.0</mechanical_reduction>
                     <offset>0.0</offset>
                 </joint>
@@ -96,5 +96,5 @@
                 <plugin>hector_transmission_interface/AdjustableOffsetTransmission</plugin>
                 <joint name="elbow" role="joint1">
-                    <mechanical_reduction>-3.0</mechanical_reduction>
+                    <mechanical_reduction>-1.0</mechanical_reduction>
                     <offset>0.0</offset>
                 </joint>

File: software/ros_ws/src/payloads/config/arm_model.urdf (robot description, URDF)
Before this commit: robot arm, 11 links, 10 joints
Joints:
- joint shoulder_pan: limit lower=-3.14159 upper=3.14159 effort=10.0 velocity=2.0 -> effort=10.0 velocity=2.0; type revolute -> continuous

Commit message: feat: integrate hector transmission interface

File: software/ros_ws/src/payloads/config/arm.ros2_control.xacro (robot description, xacro)
@@ -11,6 +11,4 @@
                   <plugin>${hardware_plugin}</plugin>
                   <param name="device">${device}</param>
-                  <!-- A 6-servo read plus write at 57600 does not fit the 100 Hz
-                       controller_manager budget; at 1 Mbaud it does. -->
                   <param name="baud_rate">1000000</param>
                   <!-- Servo IDs simulated in software rather than addressed on
@@ -62,7 +60,5 @@
             <joint name="left_finger_joint">
                 <param name="servo_id">6</param>
-                <!-- Metres of finger travel per radian of servo 6. Placeholder:
-                     15 mm over a quarter turn. Measure with the offset in
-                     left_finger_drive before un-mocking servo 6. -->
+                <!-- Metres of finger travel per radian of servo 6. Placeholder: Measure with the offset in left_finger_drive before un-mocking servo 6. -->
                 <param name="prismatic_scale">0.00955</param>
                 <command_interface name="position"/>

File: software/ros_ws/src/payloads/config/arm_model.urdf (robot description, URDF)
Before this commit: robot arm, 11 links, 10 joints
Links:
- link forearm_tip: geometry collision sphere radius=0.01; visual sphere radius=0.01
- link plate: mass 0.5 -> None

Commit message: fix(payloads): swap wrist pitch/roll channels in the differential model
On the physical wrist, co-rotation of servos 4 and 5 rolls the wrist and
counter-rotation pitches it, the opposite of the DifferentialTransmission
model: wrist_pitch rode the sum channel and wrist_roll the difference, so
commanding one joint produced the other's motion.

Swap the transmission roles (wrist_roll is joint1, wrist_pitch is joint2)
and the matching servo_id params (roll 4, pitch 5), since the hardware
plugin derives actuator1/actuator2 servo IDs from the joints holding the
joint1/joint2 roles. actuator1 remains physical servo 4 and actuator2
servo 5; each joint now commands the servo motion pattern the other used
before, with signs unchanged.

File: software/ros_ws/src/payloads/config/arm.ros2_control.xacro (robot description, xacro)
@@ -42,5 +42,5 @@
             </joint>
             <joint name="wrist_pitch">
-                <param name="servo_id">4</param>
+                <param name="servo_id">5</param>
                 <command_interface name="position"/>
                 <state_interface name="position">
@@ -50,5 +50,5 @@
             </joint>
             <joint name="wrist_roll">
-                <param name="servo_id">5</param>
+                <param name="servo_id">4</param>
                 <command_interface name="position"/>
                 <state_interface name="position">
@@ -110,12 +110,14 @@
                 </actuator>
             </transmission>
-            <!-- Servos 4 and 5 jointly drive pitch and roll. -->
+            <!-- Servos 4 and 5 jointly drive pitch and roll: co-rotation of the
+                 servos rolls the wrist, counter-rotation pitches it, so roll
+                 rides the sum channel and pitch the difference channel. -->
             <transmission name="wrist_differential">
                 <plugin>transmission_interface/DifferentialTransmission</plugin>
-                <joint name="wrist_pitch" role="joint1">
+                <joint name="wrist_roll" role="joint1">
                     <mechanical_reduction>1.0</mechanical_reduction>
                     <offset>0.0</offset>
                 </joint>
-                <joint name="wrist_roll" role="joint2">
+                <joint name="wrist_pitch" role="joint2">
                     <mechanical_reduction>1.0</mechanical_reduction>
                     <offset>0.0</offset>
