File: hardware/dc-motor-driver/_restore_backup_2026-09-27T23-58-20-985/dc-motor-driver.kicad_pcb (KiCad board)
At the start: 2 copper layers, 94 x 100 mm, 125 parts, among them J10 OQ0232510000G, J11 OQ0232510000G, J12 OQ0232510000G, J13 OQ0232510000G, J15 OQ0232510000G, J16 OQ0232510000G, J17 OQ0232510000G, J18 OQ0232510000G, J19 OQ0232510000G, J2 VIN, J20 OQ0232510000G, J3 DE9, J4 Conn_01x02, Q1 2N7002, Q2 2N7002, Q3 Si2371EDS, Q4 Si2371EDS, U1 DRV8874PWPR, U2 DRV8874PWPR, U3 DRV8874PWPR, U4 DRV8874PWPR, U5 DRV8874PWPR, U6 DRV8874PWPR, U7 SP3485CN, U8 SP3485CN

Commit message: V3R1 revision ready for review.
Connections:
- J2 pad MP: GND -> (no net)
Routing:
- net GND: track 90.9 -> 87.7 mm, vias 203 -> 206
- net Net-(D9-A): track 3.10 -> 0.00 mm
- net Net-(D16-A): track 3.03 -> 0.07 mm
- net VCC: vias 2 -> 3
