File: hardware/dc-motor-driver/_restore_backup_2026-09-27T23-58-20-985/dc-motor-driver.kicad_sch (KiCad schematic)
At the start: 20 parts, among them J2 VIN, J3 DE9, J4 Conn_01x02

Commit message: V3R1 revision ready for review.
Parts:
- added FID1, FID2, FID3: Fiducial, Fiducial:Fiducial_1.5mm_Mask3mm, symbol Mechanical:Fiducial
Other:
- note added: "Fiducial for PNP"
