File: hardware/SPACE-RESOURCES-CONTROL/power_sense.kicad_sch (KiCad schematic)
At the start: 17 parts, among them Q1 CSD19502Q5B, Q2 CSD19502Q5B, U1 LTC4368CMS-1-PBF, U2 INA238

Commit message: changed dimensions to w x l = 98.9 x 72mm, changed PCB stackup to regular (no add. copper)
Changed lines of the file:
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@@
 		)
 	)
-	(text_box "OVLO = 36V\nUVLO = 7V\nRPP = -40V\nI_{FUSE} = 20A\nI_{Inrush} = 2A @ 972uF \nt_{cooldown} = 1.2s (OC FAULT)"
+	(text_box "OVLO = 36V\nUVLO = 7V\nRPP (down to) = -40V\nI_{FUSE} = 20A\nI_{Inrush} = 2A @ 972uF \nt_{cooldown} = 1.2s (OC FAULT)"
 		(exclude_from_sim no)
 		(at 66.04 81.0786 0)
