File: hardware/SPACE-RESOURCES-CONTROL/space-resources.kicad_sch (KiCad schematic)
At the start: 25 parts, among them J1 XT90 IN, J11 OQ0232510000G, J13 OQ0232510000G, J14 OQ0232510000G, J15 OQ0232510000G, J2 XT30PW-F, J3 OQ0332510000G, J4 OQ0232510000G, J6 OQ0232510000G, J9 Smol_Brain_Board

Commit message: changed dimensions to w x l = 98.9 x 72mm, changed PCB stackup to regular (no add. copper)
Other:
- note added: "TO PERSEUS (M8 SOCKET)"
- note removed: "TO PERSEUS"
Changed lines of the file:
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@@
 		)
 	)
-	(text "TO PERSEUS"
+	(text "TO PERSEUS (M8 SOCKET)"
 		(exclude_from_sim no)
 		(at 73.914 110.236 0)
@@
 		)
 	)
-	(text_box "OVLO = 36V\nUVLO = 7V\nRPP = -40V\nI_{FUSE} = 20A\nI_{Inrush} = 3A @ 972uF \nt_{cooldown} = 1.2s (OC FAULT)"
+	(text_box "OVLO = 36V\nUVLO = 7V\nRPP (down to) = -40V\nI_{FUSE} = 20A\nI_{Inrush} = 2A @ 972uF \nt_{cooldown} = 1.2s (OC FAULT)"
 		(exclude_from_sim no)
-		(at 71.12 15.24 0)
+		(at 69.85 15.24 0)
 		(size 34.29 14.1714)
 		(margins 0.9525 0.9525 0.9525 0.9525)
@@
 	(text_box "Input Capacitance:\nPROTECTION: 100uF\nESC: 660uF \nDRILL: 101uF\nSHAFT: 101uF\nSMOL-BRAIN: 10uF\nTotal: 972uF"
 		(exclude_from_sim no)
-		(at 121.92 15.24 0)
+		(at 15.24 13.97 0)
 		(size 24.13 19.05)
 		(margins 0.9525 0.9525 0.9525 0.9525)
